Commit message: polar_description: round float values

File: urdf/gtu_arm_simple.xacro (robot description, xacro)
@@ -6,7 +6,7 @@
 <link name="base_link">
   <inertial>
-    <origin rpy="0 0 0" xyz="-0.0002980762285756305 -2.3434099167235534e-14 0.062032029672008965"/>
-    <mass value="4.6095708525443"/>
-    <inertia ixx="0.009798" ixy="1.7e-05" ixz="-2.3e-05" iyy="0.006363" iyz="0.0" izz="0.014537"/>
+    <origin rpy="0 0 0" xyz="-0.0003 -0.0 0.0620"/>
+    <mass value="4.6095"/>
+    <inertia ixx="0.0098" ixy="0.0" ixz="-0.0" iyy="0.0064" iyz="0.0" izz="0.01454"/>
   </inertial>
   <visual>
@@ -26,10 +26,10 @@
 <link name="link1_1">
   <inertial>
-    <origin rpy="0 0 0" xyz="-0.00026664559304489155 0.04142853686705264 0.01398800228501125"/>
-    <mass value="5.696621742512526"/>
-    <inertia ixx="0.020531" ixy="-2e-05" ixz="-0.000102" iyy="0.025933" iyz="-0.001156" izz="0.04291"/>
-  </inertial>
-  <visual>
-    <origin rpy="0 0 0" xyz="0.000456 0.0 -0.094999"/>
+    <origin rpy="0 0 0" xyz="-0.0003 0.0414 0.0140"/>
+    <mass value="5.6966"/>
+    <inertia ixx="0.0205" ixy="-0.0" ixz="-0.0001" iyy="0.0259" iyz="-0.0012" izz="0.0429"/>
+  </inertial>
+  <visual>
+    <origin rpy="0 0 0" xyz="0.0005 0.0 -0.095"/>
     <geometry>
       <mesh filename="package://gtu_arm_simple_description/meshes/link1_1.stl"/>
@@ -38,5 +38,5 @@
   </visual>
   <collision>
-    <origin rpy="0 0 0" xyz="0.000456 0.0 -0.094999"/>
+    <origin rpy="0 0 0" xyz="0.0005 0.0 -0.095"/>
     <geometry>
       <mesh filename="package://gtu_arm_simple_description/meshes/link1_1.stl"/>
@@ -46,10 +46,10 @@
 <link name="link2_1">
   <inertial>
-    <origin rpy="0 0 0" xyz="-0.0011265793423361435 -0.010179751209976586 0.2445690931693241"/>
-    <mass value="6.303421578081501"/>
-    <inertia ixx="0.130072" ixy="-2.8e-05" ixz="0.000325" iyy="0.111856" iyz="0.024122" izz="0.038419"/>
-  </inertial>
-  <visual>
-    <origin rpy="0 0 0" xyz="0.000999 -0.063999 -0.143997"/>
+    <origin rpy="0 0 0" xyz="-0.0011 -0.0102 0.2446"/>
+    <mass value="6.3034"/>
+    <inertia ixx="0.1301" ixy="-0.0" ixz="0.0003" iyy="0.1119" iyz="0.0241" izz="0.0384"/>
+  </inertial>
+  <visual>
+    <origin rpy="0 0 0" xyz="0.0001 -0.064 -0.144"/>
     <geometry>
       <mesh filename="package://gtu_arm_simple_description/meshes/link2_1.stl"/>
@@ -58,5 +58,5 @@
   </visual>
   <collision>
-    <origin rpy="0 0 0" xyz="0.000999 -0.063999 -0.143997"/>
+    <origin rpy="0 0 0" xyz="0.001 -0.064 -0.144"/>
     <geometry>
       <mesh filename="package://gtu_arm_simple_description/meshes/link2_1.stl"/>
@@ -66,10 +66,10 @@
 <link name="link3_1">
   <inertial>
-    <origin rpy="0 0 0" xyz="0.00023076822194436665 -0.0607138014809505 0.012742679114546629"/>
-    <mass value="2.404395336728058"/>
-    <inertia ixx="0.016491" ixy="7.1e-05" ixz="1.4e-05" iyy="0.004414" iyz="-0.002775" izz="0.016368"/>
-  </inertial>
-  <visual>
-    <origin rpy="0 0 0" xyz="0.002436 0.079687 -0.586492"/>
+    <origin rpy="0 0 0" xyz="0.0002 -0.0607 0.0127"/>
+    <mass value="2.4044"/>
+    <inertia ixx="0.0165" ixy="0.0" ixz="0.0" iyy="0.0044" iyz="-0.0028" izz="0.0164"/>
+  </inertial>
+  <visual>
+    <origin rpy="0 0 0" xyz="0.0024 0.0797 -0.5865"/>
     <geometry>
       <mesh filename="package://gtu_arm_simple_description/meshes/link3_1.stl"/>
@@ -78,5 +78,5 @@
   </visual>
   <collision>
-    <origin rpy="0 0 0" xyz="0.002436 0.079687 -0.586492"/>
+    <origin rpy="0 0 0" xyz="0.0024 0.0797 -0.5865"/>
     <geometry>
       <mesh filename="package://gtu_arm_simple_description/meshes/link3_1.stl"/>
@@ -86,10 +86,10 @@
 <link name="link4_1">
   <inertial>
-    <origin rpy="0 0 0" xyz="0.0003741376455528272 -0.0778739766529073 1.9851856895014564e-06"/>
-    <mass value="1.4724336727005185"/>
-    <inertia ixx="0.005177" ixy="1.6e-05" ixz="-4e-06" iyy="0.001869" iyz="0.0" izz="0.005924"/>
-  </inertial>
-  <visual>
-    <origin rpy="0 0 0" xyz="0.001557 0.262685 -0.586496"/>
+    <origin rpy="0 0 0" xyz="0.0004 -0.0779 0.0"/>
+    <mass value="1.4724"/>
+    <inertia ixx="0.0052" ixy="0.0" ixz="-0.0" iyy="0.0019" iyz="0.0" izz="0.0059"/>
+  </inertial>
+  <visual>
+    <origin rpy="0 0 0" xyz="0.0016 0.2627 -0.5865"/>
     <geometry>
       <mesh filename="package://gtu_arm_simple_description/meshes/link4_1.stl"/>
@@ -98,5 +98,5 @@
   </visual>
   <collision>
-    <origin rpy="0 0 0" xyz="0.001557 0.262685 -0.586496"/>
+    <origin rpy="0 0 0" xyz="0.0016 0.2627 -0.5865"/>
     <geometry>
       <mesh filename="package://gtu_arm_simple_description/meshes/link4_1.stl"/>
@@ -106,10 +106,10 @@
 <link name="link5_1">
   <inertial>
-    <origin rpy="0 0 0" xyz="0.01138398045945762 5.275851314823221e-05 -0.058028486550418146"/>
-    <mass value="2.2806063152886935"/>
-    <inertia ixx="0.011184" ixy="-1.3e-05" ixz="-0.001436" iyy="0.013878" iyz="-7e-06" izz="0.003968"/>
-  </inertial>
-  <visual>
-    <origin rpy="0 0 0" xyz="0.000829 0.414183 -0.5865"/>
+    <origin rpy="0 0 0" xyz="0.0114 0.0 -0.058"/>
+    <mass value="2.2806"/>
+    <inertia ixx="0.0112" ixy="-0.0" ixz="-0.0014" iyy="0.0139" iyz="-0.0" izz="0.004"/>
+  </inertial>
+  <visual>
+    <origin rpy="0 0 0" xyz="0.0008 0.4142 -0.5865"/>
     <geometry>
       <mesh filename="package://gtu_arm_simple_description/meshes/link5_1.stl"/>
@@ -118,5 +118,5 @@
   </visual>
   <collision>
-    <origin rpy="0 0 0" xyz="0.000829 0.414183 -0.5865"/>
+    <origin rpy="0 0 0" xyz="0.0008 0.4142 -0.5865"/>
     <geometry>
       <mesh filename="package://gtu_arm_simple_description/meshes/link5_1.stl"/>
@@ -126,10 +126,10 @@
 <link name="hand_1">
   <inertial>
-    <origin rpy="0 0 0" xyz="-4.816417538270712e-05 0.0003203293157266751 -0.036693276746967096"/>
-    <mass value="0.5768724450250841"/>
-    <inertia ixx="0.000299" ixy="1e-06" ixz="-2e-06" iyy="0.000388" iyz="4e-06" izz="0.000157"/>
-  </inertial>
-  <visual>
-    <origin rpy="0 0 0" xyz="-4e-06 0.414184 -0.413002"/>
+    <origin rpy="0 0 0" xyz="0.0 0.0003 -0.0367"/>
+    <mass value="0.5769"/>
+    <inertia ixx="0.0003" ixy="0.0" ixz="-0.0" iyy="0.0004" iyz="0.0" izz="0.0002"/>
+  </inertial>
+  <visual>
+    <origin rpy="0 0 0" xyz="0.0 0.4142 -0.413"/>
     <geometry>
       <mesh filename="package://gtu_arm_simple_description/meshes/hand_1.stl"/>
@@ -138,5 +138,5 @@
   </visual>
   <collision>
-    <origin rpy="0 0 0" xyz="-4e-06 0.414184 -0.413002"/>
+    <origin rpy="0 0 0" xyz="0.0 0.4142 -0.413"/>
     <geometry>
       <mesh filename="package://gtu_arm_simple_description/meshes/hand_1.stl"/>
@@ -146,10 +146,10 @@
 <link name="finger_r_1">
   <inertial>
-    <origin rpy="0 0 0" xyz="-0.003343915161192321 0.0035196532707398864 -0.05984017452462531"/>
-    <mass value="0.38108965550166884"/>
-    <inertia ixx="0.000418" ixy="-0.0" ixz="-2.7e-05" iyy="0.00042" iyz="-0.0" izz="7.2e-05"/>
-  </inertial>
-  <visual>
-    <origin rpy="0 0 0" xyz="0.013687 0.417713 -0.352135"/>
+    <origin rpy="0 0 0" xyz="-0.0033 0.0035 -0.0598"/>
+    <mass value="0.3811"/>
+    <inertia ixx="0.0004" ixy="-0.0" ixz="-0.0" iyy="0.0004" iyz="-0.0" izz="0.0"/>
+  </inertial>
+  <visual>
+    <origin rpy="0 0 0" xyz="0.0137 0.4177 -0.3521"/>
     <geometry>
       <mesh filename="package://gtu_arm_simple_description/meshes/finger_r_1.stl"/>
@@ -158,5 +158,5 @@
   </visual>
   <collision>
-    <origin rpy="0 0 0" xyz="0.013687 0.417713 -0.352135"/>
+    <origin rpy="0 0 0" xyz="0.0137 0.4177 -0.3521"/>
     <geometry>
       <mesh filename="package://gtu_arm_simple_description/meshes/finger_r_1.stl"/>
@@ -166,10 +166,10 @@
 <link name="finger_l_1">
   <inertial>
-    <origin rpy="0 0 0" xyz="0.0038752423274062003 0.0035783934758446545 -0.05953621179541729"/>
-    <mass value="0.3830052180747286"/>
-    <inertia ixx="0.000423" ixy="0.0" ixz="3e-05" iyy="0.000426" iyz="-0.0" izz="7.2e-05"/>
-  </inertial>
-  <visual>
-    <origin rpy="0 0 0" xyz="-0.014313 0.417617 -0.35227"/>
+    <origin rpy="0 0 0" xyz="0.0039 0.0036 -0.0595"/>
+    <mass value="0.383"/>
+    <inertia ixx="0.0004" ixy="0.0" ixz="0.0" iyy="0.0004" iyz="-0.0" izz="0.0"/>
+  </inertial>
+  <visual>
+    <origin rpy="0 0 0" xyz="-0.0143 0.4176 -0.3523"/>
     <geometry>
       <mesh filename="package://gtu_arm_simple_description/meshes/finger_l_1.stl"/>
@@ -178,5 +178,5 @@
   </visual>
   <collision>
-    <origin rpy="0 0 0" xyz="-0.014313 0.417617 -0.35227"/>
+    <origin rpy="0 0 0" xyz="-0.0143 0.4176 -0.3522"/>
     <geometry>
       <mesh filename="package://gtu_arm_simple_description/meshes/finger_l_1.stl"/>
@@ -185,50 +185,50 @@
 </link>
 <joint name="Rev1" type="continuous">
-  <origin rpy="0 0 0" xyz="-0.000456 0.0 0.094999"/>
+  <origin rpy="0 0 0" xyz="-0.0005 0.0 0.095"/>
   <parent link="base_link"/>
   <child link="link1_1"/>
-  <axis xyz="-0.004805 0.0 0.999988"/>
+  <axis xyz="-0.0048 0.0 1.0"/>
 </joint>
 <joint name="Rev2" type="continuous">
-  <origin rpy="0 0 0" xyz="-0.000543 0.063999 0.048998"/>
+  <origin rpy="0 0 0" xyz="-0.0005 0.064 0.049"/>
   <parent link="link1_1"/>
   <child link="link2_1"/>
-  <axis xyz="-0.999977 -0.004802 -0.004805"/>
+  <axis xyz="-1.0 -0.0048 -0.0048"/>
 </joint>
 <joint name="Rev3" type="continuous">
-  <origin rpy="0 0 0" xyz="-0.001437 -0.143686 0.442495"/>
+  <origin rpy="0 0 0" xyz="-0.0014 -0.1437 0.4425"/>
   <parent link="link2_1"/>
   <child link="link3_1"/>
-  <axis xyz="0.999977 0.004802 0.004805"/>
+  <axis xyz="1.0 0.0048 0.0048"/>
 </joint>
 <joint name="Rev4" type="continuous">
-  <origin rpy="0 0 0" xyz="0.000879 -0.182998 4e-06"/>
+  <origin rpy="0 0 0" xyz="0.0009 -0.1830 0.0"/>
   <parent link="link3_1"/>
   <child link="link4_1"/>
-  <axis xyz="0.004802 -0.999988 2.2e-05"/>
+  <axis xyz="0.0048 -1.0 0.0"/>
 </joint>
 <joint name="Rev5" type="continuous">
-  <origin rpy="0 0 0" xyz="0.000728 -0.151498 4e-06"/>
+  <origin rpy="0 0 0" xyz="0.0007 -0.1515 0.0"/>
   <parent link="link4_1"/>
   <child link="link5_1"/>
-  <axis xyz="0.999977 0.004802 0.004805"/>
+  <axis xyz="1.0 0.0048 0.0048"/>
 </joint>
 <joint name="Rev6" type="continuous">
-  <origin rpy="0 0 0" xyz="0.000833 -1e-06 -0.173498"/>
+  <origin rpy="0 0 0" xyz="0.0008 -0.0 -0.1735"/>
   <parent link="link5_1"/>
   <child link="hand_1"/>
-  <axis xyz="0.004805 -4e-06 -0.999988"/>
+  <axis xyz="0.0048 -0.0 -1.0"/>
 </joint>
 <joint name="Rev7" type="continuous">
-  <origin rpy="0 0 0" xyz="-0.013691 -0.003529 -0.060867"/>
+  <origin rpy="0 0 0" xyz="-0.0137 -0.0035 -0.0609"/>
   <parent link="hand_1"/>
   <child link="finger_r_1"/>
-  <axis xyz="0.004802 -0.999988 2.8e-05"/>
+  <axis xyz="0.0048 -1.0 0.0"/>
 </joint>
 <joint name="Rev8" type="continuous">
-  <origin rpy="0 0 0" xyz="0.014309 -0.003433 -0.060732"/>
+  <origin rpy="0 0 0" xyz="0.0143 -0.0034 -0.0607"/>
   <parent link="hand_1"/>
   <child link="finger_l_1"/>
-  <axis xyz="0.004802 -0.999988 2.8e-05"/>
+  <axis xyz="0.0048 -1.0 0.0"/>
 </joint>
 </robot>

Commit message: polar_description: clear mesh names

File: urdf/gtu_arm_simple.xacro (robot description, xacro)
@@ -24,5 +24,5 @@
   </collision>
 </link>
-<link name="link1_1">
+<link name="link1">
   <inertial>
     <origin rpy="0 0 0" xyz="-0.0003 0.0414 0.0140"/>
@@ -33,5 +33,5 @@
     <origin rpy="0 0 0" xyz="0.0005 0.0 -0.095"/>
     <geometry>
-      <mesh filename="package://gtu_arm_simple_description/meshes/link1_1.stl"/>
+      <mesh filename="package://gtu_arm_simple_description/meshes/link1.stl"/>
     </geometry>
     <material name="silver"/>
@@ -40,9 +40,9 @@
     <origin rpy="0 0 0" xyz="0.0005 0.0 -0.095"/>
     <geometry>
-      <mesh filename="package://gtu_arm_simple_description/meshes/link1_1.stl"/>
-    </geometry>
-  </collision>
-</link>
-<link name="link2_1">
+      <mesh filename="package://gtu_arm_simple_description/meshes/link1.stl"/>
+    </geometry>
+  </collision>
+</link>
+<link name="link2">
   <inertial>
     <origin rpy="0 0 0" xyz="-0.0011 -0.0102 0.2446"/>
@@ -53,5 +53,5 @@
     <origin rpy="0 0 0" xyz="0.0001 -0.064 -0.144"/>
     <geometry>
-      <mesh filename="package://gtu_arm_simple_description/meshes/link2_1.stl"/>
+      <mesh filename="package://gtu_arm_simple_description/meshes/link2.stl"/>
     </geometry>
     <material name="silver"/>
@@ -60,9 +60,9 @@
     <origin rpy="0 0 0" xyz="0.001 -0.064 -0.144"/>
     <geometry>
-      <mesh filename="package://gtu_arm_simple_description/meshes/link2_1.stl"/>
-    </geometry>
-  </collision>
-</link>
-<link name="link3_1">
+      <mesh filename="package://gtu_arm_simple_description/meshes/link2.stl"/>
+    </geometry>
+  </collision>
+</link>
+<link name="link3">
   <inertial>
     <origin rpy="0 0 0" xyz="0.0002 -0.0607 0.0127"/>
@@ -73,5 +73,5 @@
     <origin rpy="0 0 0" xyz="0.0024 0.0797 -0.5865"/>
     <geometry>
-      <mesh filename="package://gtu_arm_simple_description/meshes/link3_1.stl"/>
+      <mesh filename="package://gtu_arm_simple_description/meshes/link3.stl"/>
     </geometry>
     <material name="silver"/>
@@ -80,9 +80,9 @@
     <origin rpy="0 0 0" xyz="0.0024 0.0797 -0.5865"/>
     <geometry>
-      <mesh filename="package://gtu_arm_simple_description/meshes/link3_1.stl"/>
-    </geometry>
-  </collision>
-</link>
-<link name="link4_1">
+      <mesh filename="package://gtu_arm_simple_description/meshes/link3.stl"/>
+    </geometry>
+  </collision>
+</link>
+<link name="link4">
   <inertial>
     <origin rpy="0 0 0" xyz="0.0004 -0.0779 0.0"/>
@@ -93,5 +93,5 @@
     <origin rpy="0 0 0" xyz="0.0016 0.2627 -0.5865"/>
     <geometry>
-      <mesh filename="package://gtu_arm_simple_description/meshes/link4_1.stl"/>
+      <mesh filename="package://gtu_arm_simple_description/meshes/link4.stl"/>
     </geometry>
     <material name="silver"/>
@@ -100,9 +100,9 @@
     <origin rpy="0 0 0" xyz="0.0016 0.2627 -0.5865"/>
     <geometry>
-      <mesh filename="package://gtu_arm_simple_description/meshes/link4_1.stl"/>
-    </geometry>
-  </collision>
-</link>
-<link name="link5_1">
+      <mesh filename="package://gtu_arm_simple_description/meshes/link4.stl"/>
+    </geometry>
+  </collision>
+</link>
+<link name="link5">
   <inertial>
     <origin rpy="0 0 0" xyz="0.0114 0.0 -0.058"/>
@@ -113,5 +113,5 @@
     <origin rpy="0 0 0" xyz="0.0008 0.4142 -0.5865"/>
     <geometry>
-      <mesh filename="package://gtu_arm_simple_description/meshes/link5_1.stl"/>
+      <mesh filename="package://gtu_arm_simple_description/meshes/link5.stl"/>
     </geometry>
     <material name="silver"/>
@@ -120,9 +120,9 @@
     <origin rpy="0 0 0" xyz="0.0008 0.4142 -0.5865"/>
     <geometry>
-      <mesh filename="package://gtu_arm_simple_description/meshes/link5_1.stl"/>
-    </geometry>
-  </collision>
-</link>
-<link name="hand_1">
+      <mesh filename="package://gtu_arm_simple_description/meshes/link5.stl"/>
+    </geometry>
+  </collision>
+</link>
+<link name="hand">
   <inertial>
     <origin rpy="0 0 0" xyz="0.0 0.0003 -0.0367"/>
@@ -133,5 +133,5 @@
     <origin rpy="0 0 0" xyz="0.0 0.4142 -0.413"/>
     <geometry>
-      <mesh filename="package://gtu_arm_simple_description/meshes/hand_1.stl"/>
+      <mesh filename="package://gtu_arm_simple_description/meshes/hand.stl"/>
     </geometry>
     <material name="silver"/>
@@ -140,9 +140,9 @@
     <origin rpy="0 0 0" xyz="0.0 0.4142 -0.413"/>
     <geometry>
-      <mesh filename="package://gtu_arm_simple_description/meshes/hand_1.stl"/>
-    </geometry>
-  </collision>
-</link>
-<link name="finger_r_1">
+      <mesh filename="package://gtu_arm_simple_description/meshes/hand.stl"/>
+    </geometry>
+  </collision>
+</link>
+<link name="finger_r">
   <inertial>
     <origin rpy="0 0 0" xyz="-0.0033 0.0035 -0.0598"/>
@@ -153,5 +153,5 @@
     <origin rpy="0 0 0" xyz="0.0137 0.4177 -0.3521"/>
     <geometry>
-      <mesh filename="package://gtu_arm_simple_description/meshes/finger_r_1.stl"/>
+      <mesh filename="package://gtu_arm_simple_description/meshes/finger_r.stl"/>
     </geometry>
     <material name="silver"/>
@@ -160,9 +160,9 @@
     <origin rpy="0 0 0" xyz="0.0137 0.4177 -0.3521"/>
     <geometry>
-      <mesh filename="package://gtu_arm_simple_description/meshes/finger_r_1.stl"/>
-    </geometry>
-  </collision>
-</link>
-<link name="finger_l_1">
+      <mesh filename="package://gtu_arm_simple_description/meshes/finger_r.stl"/>
+    </geometry>
+  </collision>
+</link>
+<link name="finger_l">
   <inertial>
     <origin rpy="0 0 0" xyz="0.0039 0.0036 -0.0595"/>
@@ -173,5 +173,5 @@
     <origin rpy="0 0 0" xyz="-0.0143 0.4176 -0.3523"/>
     <geometry>
-      <mesh filename="package://gtu_arm_simple_description/meshes/finger_l_1.stl"/>
+      <mesh filename="package://gtu_arm_simple_description/meshes/finger_l.stl"/>
     </geometry>
     <material name="silver"/>
@@ -180,5 +180,5 @@
     <origin rpy="0 0 0" xyz="-0.0143 0.4176 -0.3522"/>
     <geometry>
-      <mesh filename="package://gtu_arm_simple_description/meshes/finger_l_1.stl"/>
+      <mesh filename="package://gtu_arm_simple_description/meshes/finger_l.stl"/>
     </geometry>
   </collision>
@@ -187,47 +187,47 @@
   <origin rpy="0 0 0" xyz="-0.0005 0.0 0.095"/>
   <parent link="base_link"/>
-  <child link="link1_1"/>
+  <child link="link1"/>
   <axis xyz="-0.0048 0.0 1.0"/>
 </joint>
 <joint name="Rev2" type="continuous">
   <origin rpy="0 0 0" xyz="-0.0005 0.064 0.049"/>
-  <parent link="link1_1"/>
-  <child link="link2_1"/>
+  <parent link="link1"/>
+  <child link="link2"/>
   <axis xyz="-1.0 -0.0048 -0.0048"/>
 </joint>
 <joint name="Rev3" type="continuous">
   <origin rpy="0 0 0" xyz="-0.0014 -0.1437 0.4425"/>
-  <parent link="link2_1"/>
-  <child link="link3_1"/>
+  <parent link="link2"/>
+  <child link="link3"/>
   <axis xyz="1.0 0.0048 0.0048"/>
 </joint>
 <joint name="Rev4" type="continuous">
   <origin rpy="0 0 0" xyz="0.0009 -0.1830 0.0"/>
-  <parent link="link3_1"/>
-  <child link="link4_1"/>
+  <parent link="link3"/>
+  <child link="link4"/>
   <axis xyz="0.0048 -1.0 0.0"/>
 </joint>
 <joint name="Rev5" type="continuous">
   <origin rpy="0 0 0" xyz="0.0007 -0.1515 0.0"/>
-  <parent link="link4_1"/>
-  <child link="link5_1"/>
+  <parent link="link4"/>
+  <child link="link5"/>
   <axis xyz="1.0 0.0048 0.0048"/>
 </joint>
 <joint name="Rev6" type="continuous">
   <origin rpy="0 0 0" xyz="0.0008 -0.0 -0.1735"/>
-  <parent link="link5_1"/>
-  <child link="hand_1"/>
+  <parent link="link5"/>
+  <child link="hand"/>
   <axis xyz="0.0048 -0.0 -1.0"/>
 </joint>
 <joint name="Rev7" type="continuous">
   <origin rpy="0 0 0" xyz="-0.0137 -0.0035 -0.0609"/>
-  <parent link="hand_1"/>
-  <child link="finger_r_1"/>
+  <parent link="hand"/>
+  <child link="finger_r"/>
   <axis xyz="0.0048 -1.0 0.0"/>
 </joint>
 <joint name="Rev8" type="continuous">
   <origin rpy="0 0 0" xyz="0.0143 -0.0034 -0.0607"/>
-  <parent link="hand_1"/>
-  <child link="finger_l_1"/>
+  <parent link="hand"/>
+  <child link="finger_l"/>
   <axis xyz="0.0048 -1.0 0.0"/>
 </joint>
