Commit message: polar_description: rename package

File: urdf/gtu_arm_simple.xacro (robot description, xacro)
@@ -1,7 +1,7 @@
 <?xml version="1.0" ?>
-<robot name="gtu_arm_simple" xmlns:xacro="http://www.ros.org/wiki/xacro">
-<xacro:include filename="$(find gtu_arm_simple_description)/urdf/materials.xacro" />
-<xacro:include filename="$(find gtu_arm_simple_description)/urdf/gtu_arm_simple.trans" />
-<xacro:include filename="$(find gtu_arm_simple_description)/urdf/gtu_arm_simple.gazebo" />
+<robot name="gtu_polar_arm" xmlns:xacro="http://www.ros.org/wiki/xacro">
+<xacro:include filename="$(find gtu_polar_arm_description)/urdf/materials.xacro" />
+<xacro:include filename="$(find gtu_polar_arm_description)/urdf/gtu_polar_arm.trans" />
+<xacro:include filename="$(find gtu_polar_arm_description)/urdf/gtu_polar_arm.gazebo" />
 <link name="base_link">
   <inertial>
@@ -13,5 +13,5 @@
     <origin rpy="0 0 0" xyz="0 0 0"/>
     <geometry>
-      <mesh filename="package://gtu_arm_simple_description/meshes/base_link.stl"/>
+      <mesh filename="package://gtu_polar_arm_description/meshes/base_link.stl"/>
     </geometry>
     <material name="silver"/>
@@ -20,5 +20,5 @@
     <origin rpy="0 0 0" xyz="0 0 0"/>
     <geometry>
-      <mesh filename="package://gtu_arm_simple_description/meshes/base_link.stl"/>
+      <mesh filename="package://gtu_polar_arm_description/meshes/base_link.stl"/>
     </geometry>
   </collision>
@@ -33,5 +33,5 @@
     <origin rpy="0 0 0" xyz="0.0005 0.0 -0.095"/>
     <geometry>
-      <mesh filename="package://gtu_arm_simple_description/meshes/link1.stl"/>
+      <mesh filename="package://gtu_polar_arm_description/meshes/link1.stl"/>
     </geometry>
     <material name="silver"/>
@@ -40,5 +40,5 @@
     <origin rpy="0 0 0" xyz="0.0005 0.0 -0.095"/>
     <geometry>
-      <mesh filename="package://gtu_arm_simple_description/meshes/link1.stl"/>
+      <mesh filename="package://gtu_polar_arm_description/meshes/link1.stl"/>
     </geometry>
   </collision>
@@ -53,5 +53,5 @@
     <origin rpy="0 0 0" xyz="0.0001 -0.064 -0.144"/>
     <geometry>
-      <mesh filename="package://gtu_arm_simple_description/meshes/link2.stl"/>
+      <mesh filename="package://gtu_polar_arm_description/meshes/link2.stl"/>
     </geometry>
     <material name="silver"/>
@@ -60,5 +60,5 @@
     <origin rpy="0 0 0" xyz="0.001 -0.064 -0.144"/>
     <geometry>
-      <mesh filename="package://gtu_arm_simple_description/meshes/link2.stl"/>
+      <mesh filename="package://gtu_polar_arm_description/meshes/link2.stl"/>
     </geometry>
   </collision>
@@ -73,5 +73,5 @@
     <origin rpy="0 0 0" xyz="0.0024 0.0797 -0.5865"/>
     <geometry>
-      <mesh filename="package://gtu_arm_simple_description/meshes/link3.stl"/>
+      <mesh filename="package://gtu_polar_arm_description/meshes/link3.stl"/>
     </geometry>
     <material name="silver"/>
@@ -80,5 +80,5 @@
     <origin rpy="0 0 0" xyz="0.0024 0.0797 -0.5865"/>
     <geometry>
-      <mesh filename="package://gtu_arm_simple_description/meshes/link3.stl"/>
+      <mesh filename="package://gtu_polar_arm_description/meshes/link3.stl"/>
     </geometry>
   </collision>
@@ -93,5 +93,5 @@
     <origin rpy="0 0 0" xyz="0.0016 0.2627 -0.5865"/>
     <geometry>
-      <mesh filename="package://gtu_arm_simple_description/meshes/link4.stl"/>
+      <mesh filename="package://gtu_polar_arm_description/meshes/link4.stl"/>
     </geometry>
     <material name="silver"/>
@@ -100,5 +100,5 @@
     <origin rpy="0 0 0" xyz="0.0016 0.2627 -0.5865"/>
     <geometry>
-      <mesh filename="package://gtu_arm_simple_description/meshes/link4.stl"/>
+      <mesh filename="package://gtu_polar_arm_description/meshes/link4.stl"/>
     </geometry>
   </collision>
@@ -113,5 +113,5 @@
     <origin rpy="0 0 0" xyz="0.0008 0.4142 -0.5865"/>
     <geometry>
-      <mesh filename="package://gtu_arm_simple_description/meshes/link5.stl"/>
+      <mesh filename="package://gtu_polar_arm_description/meshes/link5.stl"/>
     </geometry>
     <material name="silver"/>
@@ -120,5 +120,5 @@
     <origin rpy="0 0 0" xyz="0.0008 0.4142 -0.5865"/>
     <geometry>
-      <mesh filename="package://gtu_arm_simple_description/meshes/link5.stl"/>
+      <mesh filename="package://gtu_polar_arm_description/meshes/link5.stl"/>
     </geometry>
   </collision>
@@ -133,5 +133,5 @@
     <origin rpy="0 0 0" xyz="0.0 0.4142 -0.413"/>
     <geometry>
-      <mesh filename="package://gtu_arm_simple_description/meshes/hand.stl"/>
+      <mesh filename="package://gtu_polar_arm_description/meshes/hand.stl"/>
     </geometry>
     <material name="silver"/>
@@ -140,5 +140,5 @@
     <origin rpy="0 0 0" xyz="0.0 0.4142 -0.413"/>
     <geometry>
-      <mesh filename="package://gtu_arm_simple_description/meshes/hand.stl"/>
+      <mesh filename="package://gtu_polar_arm_description/meshes/hand.stl"/>
     </geometry>
   </collision>
@@ -153,5 +153,5 @@
     <origin rpy="0 0 0" xyz="0.0137 0.4177 -0.3521"/>
     <geometry>
-      <mesh filename="package://gtu_arm_simple_description/meshes/finger_r.stl"/>
+      <mesh filename="package://gtu_polar_arm_description/meshes/finger_r.stl"/>
     </geometry>
     <material name="silver"/>
@@ -160,5 +160,5 @@
     <origin rpy="0 0 0" xyz="0.0137 0.4177 -0.3521"/>
     <geometry>
-      <mesh filename="package://gtu_arm_simple_description/meshes/finger_r.stl"/>
+      <mesh filename="package://gtu_polar_arm_description/meshes/finger_r.stl"/>
     </geometry>
   </collision>
@@ -173,5 +173,5 @@
     <origin rpy="0 0 0" xyz="-0.0143 0.4176 -0.3523"/>
     <geometry>
-      <mesh filename="package://gtu_arm_simple_description/meshes/finger_l.stl"/>
+      <mesh filename="package://gtu_polar_arm_description/meshes/finger_l.stl"/>
     </geometry>
     <material name="silver"/>
@@ -180,5 +180,5 @@
     <origin rpy="0 0 0" xyz="-0.0143 0.4176 -0.3522"/>
     <geometry>
-      <mesh filename="package://gtu_arm_simple_description/meshes/finger_l.stl"/>
+      <mesh filename="package://gtu_polar_arm_description/meshes/finger_l.stl"/>
     </geometry>
   </collision>

File: urdf/materials.xacro (robot description, xacro)
@@ -1,4 +1,4 @@
 <?xml version="1.0" ?>
-<robot name="gtu_arm_simple" xmlns:xacro="http://www.ros.org/wiki/xacro" >
+<robot name="gtu_polar_arm" xmlns:xacro="http://www.ros.org/wiki/xacro" >
 <material name="silver">
   <color rgba="0.700 0.700 0.700 1.000"/>
