Commit message: polar_description: add link6, gripper

File: robots/gtu_polar_arm.xacro (robot description, xacro)
@@ -135,4 +135,26 @@
       <limit effort="12" lower="-2.8973" upper="2.8973" velocity="2.6100"/>
     </joint>
+    <link name="${arm_id}_link6">
+      <visual>
+        <origin rpy="0 0 0" xyz="0.0 0.4142 -0.4235"/>
+        <geometry>
+          <mesh filename="package://${description_pkg}/meshes/link6.dae"/>
+        </geometry>
+      </visual>
+      <collision>
+        <origin rpy="0 0 0" xyz="0.0 0.4142 -0.4235"/>
+        <geometry>
+          <mesh filename="package://${description_pkg}/meshes/link6.dae"/>
+        </geometry>
+      </collision>
+    </link>
+    <joint name="${arm_id}_joint6" type="revolute">
+      <safety_controller k_position="100.0" k_velocity="40.0" soft_lower_limit="-2.8973" soft_upper_limit="2.8973"/>
+      <origin rpy="0 0 0" xyz="0.0008 -0.0 -0.1630"/>
+      <parent link="${arm_id}_link5"/>
+      <child link="${arm_id}_link6"/>
+      <axis xyz="0.0048 -0.0 -1.0"/>
+      <limit effort="12" lower="-2.8973" upper="2.8973" velocity="2.6100"/>
+    </joint>
   </xacro:macro>
 </robot>

File: robots/gtu_polar_arm_hand.urdf.xacro (robot description, xacro)
@@ -4,4 +4,5 @@
   <xacro:include filename="$(find gtu_polar_arm_description)/robots/hand.xacro"/>
   <xacro:gtu_polar_arm/>
-  <xacro:hand ns="gtu_polar" connected_to="gtu_polar_link5"/>
+  <!-- <xacro:hand ns="gtu_polar" rpy="0 0 0" xyz="0.0008 -0.0 -0.1735" connected_to="gtu_polar_link5"/> -->
+  <xacro:hand ns="gtu_polar" rpy="${pi/2} 0 0" xyz="-0.00675 -0.00964 -0.06152" connected_to="gtu_polar_link6"/>
 </robot>

File: robots/hand.xacro (robot description, xacro)
@@ -12,58 +12,99 @@
     <link name="${ns}_hand">
       <visual>
-        <origin rpy="0 0 0" xyz="0.0 0.4142 -0.413"/>
+        <origin rpy="0 0 0" xyz="0 0 0"/>
         <geometry>
-          <mesh filename="package://gtu_polar_arm_description/meshes/hand.stl"/>
+          <mesh filename="package://gtu_polar_arm_description/meshes/gripper/hand.dae"/>
         </geometry>
       </visual>
       <collision>
-        <origin rpy="0 0 0" xyz="0.0 0.4142 -0.413"/>
+        <origin rpy="0 0 0" xyz="0 0 0"/>
         <geometry>
-          <mesh filename="package://gtu_polar_arm_description/meshes/hand.stl"/>
+          <mesh filename="package://gtu_polar_arm_description/meshes/gripper/hand.dae"/>
         </geometry>
       </collision>
     </link>
-    <link name="${ns}_leftfinger">
+    <link name="${ns}_outer_r">
       <visual>
-        <origin rpy="0 0 0" xyz="-0.0143 0.4176 -0.3523"/>
+        <origin rpy="0 0 0" xyz="0.011889 0.027594 0.004951"/>
         <geometry>
-          <mesh filename="package://gtu_polar_arm_description/meshes/finger_l.stl"/>
+          <mesh filename="package://gtu_polar_arm_description/meshes/gripper/outer_r.dae"/>
         </geometry>
       </visual>
-      <!-- <collision>
-        <origin rpy="0 0 0" xyz="-0.0143 0.4176 -0.3523"/>
+      <collision>
+        <origin rpy="0 0 0" xyz="0.011889 0.027594 0.004951"/>
         <geometry>
-          <mesh filename="package://gtu_polar_arm_description/meshes/finger.stl"/>
+          <mesh filename="package://gtu_polar_arm_description/meshes/gripper/outer_r.dae"/>
         </geometry>
-      </collision> -->
+      </collision>
     </link>
-    <link name="${ns}_rightfinger">
+    <link name="${ns}_outer_l">
       <visual>
-        <origin rpy="0 0 0" xyz="0.0137 0.4177 -0.3521"/>
+        <origin rpy="0 0 0" xyz="-0.025351 0.027594 0.004951"/>
         <geometry>
-          <mesh filename="package://gtu_polar_arm_description/meshes/finger_r.stl"/>
+          <mesh filename="package://gtu_polar_arm_description/meshes/gripper/outer_l.dae"/>
         </geometry>
       </visual>
-      <!-- <collision>
-        <origin rpy="0 0 0" xyz="0.0137 0.4177 -0.3521"/>
+      <collision>
+        <origin rpy="0 0 0" xyz="-0.025351 0.027594 0.004951"/>
         <geometry>
-          <mesh filename="package://gtu_polar_arm_description/meshes/finger.stl"/>
+          <mesh filename="package://gtu_polar_arm_description/meshes/gripper/outer_l.dae"/>
         </geometry>
-      </collision> -->
-   </link>
-    <joint name="${ns}_finger_joint1" type="revolute">
+      </collision>
+    </link>
+    <link name="${ns}_finger_l">
+      <visual>
+        <origin rpy="0 0 0" xyz="-0.061266 0.066842 0.004951"/>
+        <geometry>
+          <mesh filename="package://gtu_polar_arm_description/meshes/gripper/finger_l.dae"/>
+        </geometry>
+      </visual>
+      <collision>
+        <origin rpy="0 0 0" xyz="-0.061266 0.066842 0.004951"/>
+        <geometry>
+          <mesh filename="package://gtu_polar_arm_description/meshes/gripper/finger_l.dae"/>
+        </geometry>
+      </collision>
+    </link>
+    <link name="${ns}_finger_r">
+      <visual>
+        <origin rpy="0 0 0" xyz="0.047804 0.066842 0.004951"/>
+        <geometry>
+          <mesh filename="package://gtu_polar_arm_description/meshes/gripper/finger_r.dae"/>
+        </geometry>
+      </visual>
+      <collision>
+        <origin rpy="0 0 0" xyz="0.047804 0.066842 0.004951"/>
+        <geometry>
+          <mesh filename="package://gtu_polar_arm_description/meshes/gripper/finger_r.dae"/>
+        </geometry>
+      </collision>
+    </link>
+    <joint name="${ns}_hand_joint2" type="continuous">
+      <origin rpy="0 0 0" xyz="-0.011889 -0.027594 -0.004951"/>
       <parent link="${ns}_hand"/>
-      <child link="${ns}_leftfinger"/>
-      <origin rpy="0 0 0" xyz="0.0143 -0.0034 -0.0607"/>
-      <axis xyz="0.0048 -1.0 0.0"/>
-      <limit effort="20" lower="0.0" upper="0.04" velocity="0.2"/>
-      <mimic joint="${ns}_finger_joint2" />
+      <child link="${ns}_outer_r"/>
+      <axis xyz="0.0 -0.0 -1.0"/>
+      <mimic joint="${ns}_hand_joint1" multiplier="-1.0"/>
     </joint>
-    <joint name="${ns}_finger_joint2" type="revolute">
+    <joint name="${ns}_hand_joint1" type="revolute">
+      <origin rpy="0 0 0" xyz="0.025351 -0.027594 -0.004951"/>
       <parent link="${ns}_hand"/>
-      <child link="${ns}_rightfinger"/>
-      <origin rpy="0 0 0" xyz="-0.0137 -0.0035 -0.0609"/>
-      <axis xyz="0.0048 -1.0 0.0"/>
-      <limit effort="20" lower="0.0" upper="0.04" velocity="0.2"/>
+      <child link="${ns}_outer_l"/>
+      <axis xyz="0.0 -0.0 -1.0"/>
+      <limit effort="100" lower="-0.827286" upper="0.74002" velocity="100"/>
+    </joint>
+    <joint name="${ns}_finger_joint1" type="continuous">
+      <origin rpy="0 0 0" xyz="0.035915 -0.039248 0.0"/>
+      <parent link="${ns}_outer_l"/>
+      <child link="${ns}_finger_l"/>
+      <axis xyz="-0.0 -0.0 -1.0"/>
+      <mimic joint="${ns}_finger_joint2"/>
+    </joint>
+    <joint name="${ns}_finger_joint2" type="continuous">
+      <origin rpy="0 0 0" xyz="-0.035915 -0.039248 0.0"/>
+      <parent link="${ns}_outer_r"/>
+      <child link="${ns}_finger_r"/>
+      <axis xyz="0.0 0.0 1.0"/>
+      <mimic joint="${ns}_hand_joint1" multiplier="-1.0"/>
     </joint>
   </xacro:macro>

Commit message: polar_description: add joint limits

File: robots/gtu_polar_arm.xacro (robot description, xacro)
@@ -40,10 +40,10 @@
     </link>
     <joint name="${arm_id}_joint1" type="revolute">
-      <safety_controller k_position="100.0" k_velocity="40.0" soft_lower_limit="-2.8973" soft_upper_limit="2.8973"/>
+      <safety_controller k_position="100.0" k_velocity="40.0" soft_lower_limit="${-1.2*pi}" soft_upper_limit="${1.2*pi}"/>
       <origin rpy="0 0 0" xyz="-0.0005 0.0 0.095"/>
       <parent link="${arm_id}_link0"/>
       <child link="${arm_id}_link1"/>
       <axis xyz="-0.0048 0.0 1.0"/>
-      <limit effort="87" lower="-2.8973" upper="2.8973" velocity="2.1750"/>
+      <limit effort="87" lower="${-1.2*pi}" upper="${1.2*pi}" velocity="2.1750"/>
     </joint>
     <link name="${arm_id}_link2">
@@ -62,10 +62,10 @@
     </link>
     <joint name="${arm_id}_joint2" type="revolute">
-      <safety_controller k_position="100.0" k_velocity="40.0" soft_lower_limit="-1.7628" soft_upper_limit="1.7628"/>
+      <safety_controller k_position="100.0" k_velocity="40.0" soft_lower_limit="-0.96" soft_upper_limit="0.35"/>
       <origin rpy="0 0 0" xyz="-0.0005 0.064 0.049"/>
       <parent link="${arm_id}_link1"/>
       <child link="${arm_id}_link2"/>
       <axis xyz="-1.0 -0.0048 -0.0048"/>
-      <limit effort="87" lower="-1.7628" upper="1.7628" velocity="2.1750"/>
+      <limit effort="87" lower="-0.96" upper="0.35" velocity="2.1750"/>
     </joint>
     <link name="${arm_id}_link3">
@@ -84,10 +84,10 @@
     </link>
     <joint name="${arm_id}_joint3" type="revolute">
-      <safety_controller k_position="100.0" k_velocity="40.0" soft_lower_limit="-2.8973" soft_upper_limit="2.8973"/>
+      <safety_controller k_position="100.0" k_velocity="40.0" soft_lower_limit="-0.26" soft_upper_limit="0.87"/>
       <origin rpy="0 0 0" xyz="-0.0014 -0.1437 0.4425"/>
       <parent link="${arm_id}_link2"/>
       <child link="${arm_id}_link3"/>
       <axis xyz="1.0 0.0048 0.0048"/>
-      <limit effort="87" lower="-2.8973" upper="2.8973" velocity="2.1750"/>
+      <limit effort="87" lower="-0.26" upper="0.87" velocity="2.1750"/>
     </joint>
     <link name="${arm_id}_link4">
@@ -106,10 +106,11 @@
     </link>
     <joint name="${arm_id}_joint4" type="revolute">
-      <safety_controller k_position="100.0" k_velocity="40.0" soft_lower_limit="-3.0718" soft_upper_limit="-0.0698"/>
+      <safety_controller k_position="100.0" k_velocity="40.0" soft_lower_limit="${-pi}" soft_upper_limit="${pi}"/>
       <origin rpy="0 0 0" xyz="0.0009 -0.1830 0.0"/>
       <parent link="${arm_id}_link3"/>
       <child link="${arm_id}_link4"/>
       <axis xyz="0.0048 -1.0 0.0"/>
-      <limit effort="87" lower="-3.0718" upper="-0.0698" velocity="2.1750"/>
+      <limit effort="87" lower="${-pi}" upper="${pi}" velocity="2.1750"/>
+      <!-- gerçek değer -->
     </joint>
     <link name="${arm_id}_link5">
@@ -128,10 +129,10 @@
     </link>
     <joint name="${arm_id}_joint5" type="revolute">
-      <safety_controller k_position="100.0" k_velocity="40.0" soft_lower_limit="-2.8973" soft_upper_limit="2.8973"/>
+      <safety_controller k_position="100.0" k_velocity="40.0" soft_lower_limit="${-pi}" soft_upper_limit="0.96"/>
       <origin rpy="0 0 0" xyz="0.0007 -0.1515 0.0"/>
       <parent link="${arm_id}_link4"/>
       <child link="${arm_id}_link5"/>
       <axis xyz="1.0 0.0048 0.0048"/>
-      <limit effort="12" lower="-2.8973" upper="2.8973" velocity="2.6100"/>
+      <limit effort="12" lower="${-pi}" upper="0.96" velocity="2.6100"/>
     </joint>
     <link name="${arm_id}_link6">
@@ -150,10 +151,10 @@
     </link>
     <joint name="${arm_id}_joint6" type="revolute">
-      <safety_controller k_position="100.0" k_velocity="40.0" soft_lower_limit="-2.8973" soft_upper_limit="2.8973"/>
+      <safety_controller k_position="100.0" k_velocity="40.0" soft_lower_limit="${-pi}" soft_upper_limit="${pi}"/>
       <origin rpy="0 0 0" xyz="0.0008 -0.0 -0.1630"/>
       <parent link="${arm_id}_link5"/>
       <child link="${arm_id}_link6"/>
       <axis xyz="0.0048 -0.0 -1.0"/>
-      <limit effort="12" lower="-2.8973" upper="2.8973" velocity="2.6100"/>
+      <limit effort="12" lower="${-pi}" upper="${pi}" velocity="2.6100"/>
     </joint>
   </xacro:macro>

Commit message: polar_description: add world joint add damping, friction and safety limits

File: robots/gtu_polar_arm.xacro (robot description, xacro)
@@ -11,4 +11,14 @@
       </joint>
     </xacro:unless>
+    <xacro:property name="joint_damping" value="0.0"/>
+    <xacro:property name="joint_friction" value="0.0"/>
+    <xacro:property name="safety_k_position" value="100.0"/>
+    <xacro:property name="safety_k_velocity" value="40.0"/>
+    <link name="world" />
+    <joint name="robot_to_world" type="fixed">
+      <parent link="world" />
+      <child link="${arm_id}_link0" />
+      <origin xyz="0.0 0.0 0.0" rpy="0.0 0.0 0.0" />
+    </joint>
     <link name="${arm_id}_link0">
       <visual>
@@ -40,5 +50,5 @@
     </link>
     <joint name="${arm_id}_joint1" type="revolute">
-      <safety_controller k_position="100.0" k_velocity="40.0" soft_lower_limit="${-1.2*pi}" soft_upper_limit="${1.2*pi}"/>
+      <safety_controller k_position="${safety_k_position}" k_velocity="${safety_k_velocity}" soft_lower_limit="${-1.2*pi}" soft_upper_limit="${1.2*pi}"/>
       <origin rpy="0 0 0" xyz="-0.0005 0.0 0.095"/>
       <parent link="${arm_id}_link0"/>
@@ -46,4 +56,5 @@
       <axis xyz="-0.0048 0.0 1.0"/>
       <limit effort="87" lower="${-1.2*pi}" upper="${1.2*pi}" velocity="2.1750"/>
+      <dynamics damping="${joint_damping}" friction="${joint_friction}"/>
     </joint>
     <link name="${arm_id}_link2">
@@ -62,5 +73,5 @@
     </link>
     <joint name="${arm_id}_joint2" type="revolute">
-      <safety_controller k_position="100.0" k_velocity="40.0" soft_lower_limit="-0.96" soft_upper_limit="0.35"/>
+      <safety_controller k_position="${safety_k_position}" k_velocity="${safety_k_velocity}" soft_lower_limit="-0.96" soft_upper_limit="0.35"/>
       <origin rpy="0 0 0" xyz="-0.0005 0.064 0.049"/>
       <parent link="${arm_id}_link1"/>
@@ -68,4 +79,5 @@
       <axis xyz="-1.0 -0.0048 -0.0048"/>
       <limit effort="87" lower="-0.96" upper="0.35" velocity="2.1750"/>
+      <dynamics damping="${joint_damping}" friction="${joint_friction}"/>
     </joint>
     <link name="${arm_id}_link3">
@@ -84,5 +96,5 @@
     </link>
     <joint name="${arm_id}_joint3" type="revolute">
-      <safety_controller k_position="100.0" k_velocity="40.0" soft_lower_limit="-0.26" soft_upper_limit="0.87"/>
+      <safety_controller k_position="${safety_k_position}" k_velocity="${safety_k_velocity}" soft_lower_limit="-0.26" soft_upper_limit="0.87"/>
       <origin rpy="0 0 0" xyz="-0.0014 -0.1437 0.4425"/>
       <parent link="${arm_id}_link2"/>
@@ -90,4 +102,5 @@
       <axis xyz="1.0 0.0048 0.0048"/>
       <limit effort="87" lower="-0.26" upper="0.87" velocity="2.1750"/>
+      <dynamics damping="${joint_damping}" friction="${joint_friction}"/>
     </joint>
     <link name="${arm_id}_link4">
@@ -106,5 +119,5 @@
     </link>
     <joint name="${arm_id}_joint4" type="revolute">
-      <safety_controller k_position="100.0" k_velocity="40.0" soft_lower_limit="${-pi}" soft_upper_limit="${pi}"/>
+      <safety_controller k_position="${safety_k_position}" k_velocity="${safety_k_velocity}" soft_lower_limit="${-pi}" soft_upper_limit="${pi}"/>
       <origin rpy="0 0 0" xyz="0.0009 -0.1830 0.0"/>
       <parent link="${arm_id}_link3"/>
@@ -112,5 +125,5 @@
       <axis xyz="0.0048 -1.0 0.0"/>
       <limit effort="87" lower="${-pi}" upper="${pi}" velocity="2.1750"/>
-      <!-- gerçek değer -->
+      <dynamics damping="${joint_damping}" friction="${joint_friction}"/>
     </joint>
     <link name="${arm_id}_link5">
@@ -129,5 +142,5 @@
     </link>
     <joint name="${arm_id}_joint5" type="revolute">
-      <safety_controller k_position="100.0" k_velocity="40.0" soft_lower_limit="${-pi}" soft_upper_limit="0.96"/>
+      <safety_controller k_position="${safety_k_position}" k_velocity="${safety_k_velocity}" soft_lower_limit="${-pi}" soft_upper_limit="0.96"/>
       <origin rpy="0 0 0" xyz="0.0007 -0.1515 0.0"/>
       <parent link="${arm_id}_link4"/>
@@ -135,4 +148,5 @@
       <axis xyz="1.0 0.0048 0.0048"/>
       <limit effort="12" lower="${-pi}" upper="0.96" velocity="2.6100"/>
+      <dynamics damping="${joint_damping}" friction="${joint_friction}"/>
     </joint>
     <link name="${arm_id}_link6">
@@ -151,5 +165,5 @@
     </link>
     <joint name="${arm_id}_joint6" type="revolute">
-      <safety_controller k_position="100.0" k_velocity="40.0" soft_lower_limit="${-pi}" soft_upper_limit="${pi}"/>
+      <safety_controller k_position="${safety_k_position}" k_velocity="${safety_k_velocity}" soft_lower_limit="${-pi}" soft_upper_limit="${pi}"/>
       <origin rpy="0 0 0" xyz="0.0008 -0.0 -0.1630"/>
       <parent link="${arm_id}_link5"/>
@@ -157,4 +171,5 @@
       <axis xyz="0.0048 -0.0 -1.0"/>
       <limit effort="12" lower="${-pi}" upper="${pi}" velocity="2.6100"/>
+      <dynamics damping="${joint_damping}" friction="${joint_friction}"/>
     </joint>
   </xacro:macro>

Commit message: polar_description: add inertials

File: robots/gtu_polar_arm.xacro (robot description, xacro)
@@ -34,4 +34,9 @@
         </geometry>
       </collision>
+      <inertial>
+        <origin rpy="0 0 0" xyz="-0.0003 -0.0 0.0620"/>
+        <mass value="4.6095708525443"/>
+        <inertia ixx="0.009798" ixy="1.7e-05" ixz="-2.3e-05" iyy="0.006363" iyz="0.0" izz="0.014537"/>
+      </inertial>
     </link>
     <link name="${arm_id}_link1">
@@ -48,4 +53,9 @@
         </geometry>
       </collision>
+      <inertial>
+        <origin rpy="0 0 0" xyz="-0.00026664559304489155 0.04142853686705264 0.01398800228501125"/>
+        <mass value="5.696621742512526"/>
+        <inertia ixx="0.020531" ixy="-2e-05" ixz="-0.000102" iyy="0.025933" iyz="-0.001156" izz="0.04291"/>
+      </inertial>
     </link>
     <joint name="${arm_id}_joint1" type="revolute">
@@ -71,4 +81,9 @@
         </geometry>
       </collision>
+      <inertial>
+        <origin rpy="0 0 0" xyz="-0.0011265793423361435 -0.010179751209976586 0.2445690931693241"/>
+        <mass value="6.303421578081501"/>
+        <inertia ixx="0.130072" ixy="-2.8e-05" ixz="0.000325" iyy="0.111856" iyz="0.024122" izz="0.038419"/>
+      </inertial>
     </link>
     <joint name="${arm_id}_joint2" type="revolute">
@@ -94,4 +109,9 @@
         </geometry>
       </collision>
+      <inertial>
+        <origin rpy="0 0 0" xyz="0.00023076822194436665 -0.0607138014809505 0.012742679114546629"/>
+        <mass value="2.404395336728058"/>
+        <inertia ixx="0.016491" ixy="7.1e-05" ixz="1.4e-05" iyy="0.004414" iyz="-0.002775" izz="0.016368"/>
+      </inertial>
     </link>
     <joint name="${arm_id}_joint3" type="revolute">
@@ -117,4 +137,9 @@
         </geometry>
       </collision>
+      <inertial>
+        <origin rpy="0 0 0" xyz="0.0003741376455528272 -0.0778739766529073 1.9851856895014564e-06"/>
+        <mass value="1.4724336727005185"/>
+        <inertia ixx="0.005177" ixy="1.6e-05" ixz="-4e-06" iyy="0.001869" iyz="0.0" izz="0.005924"/>
+      </inertial>
     </link>
     <joint name="${arm_id}_joint4" type="revolute">
@@ -140,4 +165,9 @@
         </geometry>
       </collision>
+      <inertial>
+        <origin rpy="0 0 0" xyz="0.011505440232523104 5.3376606865773724e-05 -0.056762648886386935"/>
+        <mass value="2.254711737840762"/>
+        <inertia ixx="0.010865" ixy="-1.3e-05" ixz="-0.001406" iyy="0.013556" iyz="-7e-06" izz="0.003964"/>
+      </inertial>
     </link>
     <joint name="${arm_id}_joint5" type="revolute">
@@ -163,4 +193,9 @@
         </geometry>
       </collision>
+      <inertial>
+        <origin rpy="0 0 0" xyz="2.4665038927900798e-05 -6.015326359243289e-08 -0.005150438004958846"/>
+        <mass value="0.02540134740060902"/>
+        <inertia ixx="1e-06" ixy="-0.0" ixz="-0.0" iyy="1e-06" iyz="0.0" izz="1e-06"/>
+      </inertial>
     </link>
     <joint name="${arm_id}_joint6" type="revolute">

Commit message: polar_description: round arm inertials

File: robots/gtu_polar_arm.xacro (robot description, xacro)
@@ -36,6 +36,6 @@
       <inertial>
         <origin rpy="0 0 0" xyz="-0.0003 -0.0 0.0620"/>
-        <mass value="4.6095708525443"/>
-        <inertia ixx="0.009798" ixy="1.7e-05" ixz="-2.3e-05" iyy="0.006363" iyz="0.0" izz="0.014537"/>
+        <mass value="4.6096"/>
+        <inertia ixx="0.0098" ixy="0.0" ixz="-0.0" iyy="0.0064" iyz="0.0" izz="0.0145"/>
       </inertial>
     </link>
@@ -54,7 +54,7 @@
       </collision>
       <inertial>
-        <origin rpy="0 0 0" xyz="-0.00026664559304489155 0.04142853686705264 0.01398800228501125"/>
-        <mass value="5.696621742512526"/>
-        <inertia ixx="0.020531" ixy="-2e-05" ixz="-0.000102" iyy="0.025933" iyz="-0.001156" izz="0.04291"/>
+        <origin rpy="0 0 0" xyz="-0.0003 0.0414 0.0140"/>
+        <mass value="5.6966"/>
+        <inertia ixx="0.0205" ixy="-0.0" ixz="-0.0001" iyy="0.0259" iyz="-0.0012" izz="0.0429"/>
       </inertial>
     </link>
@@ -82,7 +82,7 @@
       </collision>
       <inertial>
-        <origin rpy="0 0 0" xyz="-0.0011265793423361435 -0.010179751209976586 0.2445690931693241"/>
-        <mass value="6.303421578081501"/>
-        <inertia ixx="0.130072" ixy="-2.8e-05" ixz="0.000325" iyy="0.111856" iyz="0.024122" izz="0.038419"/>
+        <origin rpy="0 0 0" xyz="-0.0011 -0.0102 0.2446"/>
+        <mass value="6.3034"/>
+        <inertia ixx="0.1301" ixy="-0.0" ixz="0.0003" iyy="0.1119" iyz="0.0241" izz="0.0384"/>
       </inertial>
     </link>
@@ -110,7 +110,7 @@
       </collision>
       <inertial>
-        <origin rpy="0 0 0" xyz="0.00023076822194436665 -0.0607138014809505 0.012742679114546629"/>
-        <mass value="2.404395336728058"/>
-        <inertia ixx="0.016491" ixy="7.1e-05" ixz="1.4e-05" iyy="0.004414" iyz="-0.002775" izz="0.016368"/>
+        <origin rpy="0 0 0" xyz="0.0002 -0.0607 0.0127"/>
+        <mass value="2.4044"/>
+        <inertia ixx="0.0165" ixy="0.0" ixz="0.0" iyy="0.0044" iyz="-0.0028" izz="0.0164"/>
       </inertial>
     </link>
@@ -138,7 +138,7 @@
       </collision>
       <inertial>
-        <origin rpy="0 0 0" xyz="0.0003741376455528272 -0.0778739766529073 1.9851856895014564e-06"/>
-        <mass value="1.4724336727005185"/>
-        <inertia ixx="0.005177" ixy="1.6e-05" ixz="-4e-06" iyy="0.001869" iyz="0.0" izz="0.005924"/>
+        <origin rpy="0 0 0" xyz="0.0004 -0.0779 0.0"/>
+        <mass value="1.4724"/>
+        <inertia ixx="0.0052" ixy="0.0" ixz="-0.0" iyy="0.0019" iyz="0.0" izz="0.0059"/>
       </inertial>
     </link>
@@ -166,7 +166,7 @@
       </collision>
       <inertial>
-        <origin rpy="0 0 0" xyz="0.011505440232523104 5.3376606865773724e-05 -0.056762648886386935"/>
-        <mass value="2.254711737840762"/>
-        <inertia ixx="0.010865" ixy="-1.3e-05" ixz="-0.001406" iyy="0.013556" iyz="-7e-06" izz="0.003964"/>
+        <origin rpy="0 0 0" xyz="0.0115 0.0 -0.0568"/>
+        <mass value="2.2547"/>
+        <inertia ixx="0.0109" ixy="-0.0" ixz="-0.0014" iyy="0.0136" iyz="-0.0" izz="0.0040"/>
       </inertial>
     </link>
@@ -194,7 +194,7 @@
       </collision>
       <inertial>
-        <origin rpy="0 0 0" xyz="2.4665038927900798e-05 -6.015326359243289e-08 -0.005150438004958846"/>
-        <mass value="0.02540134740060902"/>
-        <inertia ixx="1e-06" ixy="-0.0" ixz="-0.0" iyy="1e-06" iyz="0.0" izz="1e-06"/>
+        <origin rpy="0 0 0" xyz="0.0 0.0 -0.005"/>
+        <mass value="0.0254"/>
+        <inertia ixx="0.0" ixy="-0.0" ixz="-0.0" iyy="0.0" iyz="0.0" izz="0.0"/>
       </inertial>
     </link>
