Commit message: polar_description: add gazebo and transmission

File: robots/gtu_polar_arm_hand.urdf.xacro (robot description, xacro)
@@ -1,8 +1,12 @@
 <?xml version="1.0" encoding="utf-8"?>
 <robot xmlns:xacro="http://www.ros.org/wiki/xacro" name="gtu_polar">
+  <xacro:arg name="robot_name" default="gtu_polar"/>
   <xacro:include filename="$(find gtu_polar_arm_description)/robots/gtu_polar_arm.xacro"/>
   <xacro:include filename="$(find gtu_polar_arm_description)/robots/hand.xacro"/>
+  <xacro:include filename="$(find gtu_polar_arm_description)/robots/gtu_polar.gazebo.xacro"/>
+  <xacro:include filename="$(find gtu_polar_arm_description)/robots/gtu_polar.transmission.xacro"/>
   <xacro:gtu_polar_arm/>
-  <!-- <xacro:hand ns="gtu_polar" rpy="0 0 0" xyz="0.0008 -0.0 -0.1735" connected_to="gtu_polar_link5"/> -->
   <xacro:hand ns="gtu_polar" rpy="${pi/2} 0 0" xyz="-0.00675 -0.00964 -0.06152" connected_to="gtu_polar_link6"/>
+  <xacro:gtu_polar_gazebo robot_name="$(arg robot_name)" />
+  <xacro:gtu_polar_transmission robot_name="$(arg robot_name)" />
 </robot>

File: robots/hand.xacro (robot description, xacro)
@@ -29,4 +29,23 @@
       </inertial>
     </link>
+    <link name="${ns}_outer_l">
+      <visual>
+        <origin rpy="0 0 0" xyz="-0.025351 0.027594 0.004951"/>
+        <geometry>
+          <mesh filename="package://gtu_polar_arm_description/meshes/gripper/outer_l.dae"/>
+        </geometry>
+      </visual>
+      <collision>
+        <origin rpy="0 0 0" xyz="-0.025351 0.027594 0.004951"/>
+        <geometry>
+          <mesh filename="package://gtu_polar_arm_description/meshes/gripper/outer_l.dae"/>
+        </geometry>
+      </collision>
+      <inertial>
+        <origin rpy="0 0 0" xyz="0.006975 -0.006230 -0.004655"/>
+        <mass value="0.0877"/>
+        <inertia ixx="0.0" ixy="0.0" ixz="-0.0" iyy="0.0" iyz="0.0" izz="0.0"/>
+      </inertial>
+    </link>
     <link name="${ns}_outer_r">
       <visual>
@@ -46,23 +65,4 @@
         <mass value="0.0868"/>
         <inertia ixx="0.0" ixy="0.0" ixz="0.0" iyy="0.0" iyz="-0.0" izz="0.0"/>
-      </inertial>
-    </link>
-    <link name="${ns}_outer_l">
-      <visual>
-        <origin rpy="0 0 0" xyz="-0.025351 0.027594 0.004951"/>
-        <geometry>
-          <mesh filename="package://gtu_polar_arm_description/meshes/gripper/outer_l.dae"/>
-        </geometry>
-      </visual>
-      <collision>
-        <origin rpy="0 0 0" xyz="-0.025351 0.027594 0.004951"/>
-        <geometry>
-          <mesh filename="package://gtu_polar_arm_description/meshes/gripper/outer_l.dae"/>
-        </geometry>
-      </collision>
-      <inertial>
-        <origin rpy="0 0 0" xyz="0.006975 -0.006230 -0.004655"/>
-        <mass value="0.0877"/>
-        <inertia ixx="0.0" ixy="0.0" ixz="-0.0" iyy="0.0" iyz="0.0" izz="0.0"/>
       </inertial>
     </link>
