Commit message: polar_description: - rename package and files - delete stl files

File: robots/hand.urdf.xacro (robot description, xacro)
@@ -2,4 +2,4 @@
 <robot xmlns:xacro="http://www.ros.org/wiki/xacro" name="hand">
   <xacro:include filename="hand.xacro"/>
-  <xacro:hand ns="gtu_polar"/>
+  <xacro:hand ns="polar"/>
 </robot>

File: robots/hand.xacro (robot description, xacro)
@@ -14,5 +14,5 @@
         <origin rpy="0 0 0" xyz="0 0 0"/>
         <geometry>
-          <mesh filename="package://gtu_polar_arm_description/meshes/gripper/hand.dae"/>
+          <mesh filename="package://polar_description/meshes/gripper/hand.dae"/>
         </geometry>
       </visual>
@@ -20,5 +20,5 @@
         <origin rpy="0 0 0" xyz="0 0 0"/>
         <geometry>
-          <mesh filename="package://gtu_polar_arm_description/meshes/gripper/hand.dae"/>
+          <mesh filename="package://polar_description/meshes/gripper/hand.dae"/>
         </geometry>
       </collision>
@@ -33,5 +33,5 @@
         <origin rpy="0 0 0" xyz="-0.025351 0.027594 0.004951"/>
         <geometry>
-          <mesh filename="package://gtu_polar_arm_description/meshes/gripper/outer_l.dae"/>
+          <mesh filename="package://polar_description/meshes/gripper/outer_l.dae"/>
         </geometry>
       </visual>
@@ -39,5 +39,5 @@
         <origin rpy="0 0 0" xyz="-0.025351 0.027594 0.004951"/>
         <geometry>
-          <mesh filename="package://gtu_polar_arm_description/meshes/gripper/outer_l.dae"/>
+          <mesh filename="package://polar_description/meshes/gripper/outer_l.dae"/>
         </geometry>
       </collision>
@@ -52,5 +52,5 @@
         <origin rpy="0 0 0" xyz="0.011889 0.027594 0.004951"/>
         <geometry>
-          <mesh filename="package://gtu_polar_arm_description/meshes/gripper/outer_r.dae"/>
+          <mesh filename="package://polar_description/meshes/gripper/outer_r.dae"/>
         </geometry>
       </visual>
@@ -58,5 +58,5 @@
         <origin rpy="0 0 0" xyz="0.011889 0.027594 0.004951"/>
         <geometry>
-          <mesh filename="package://gtu_polar_arm_description/meshes/gripper/outer_r.dae"/>
+          <mesh filename="package://polar_description/meshes/gripper/outer_r.dae"/>
         </geometry>
       </collision>
@@ -71,5 +71,5 @@
         <origin rpy="0 0 0" xyz="-0.061266 0.066842 0.004951"/>
         <geometry>
-          <mesh filename="package://gtu_polar_arm_description/meshes/gripper/finger_l.dae"/>
+          <mesh filename="package://polar_description/meshes/gripper/finger_l.dae"/>
         </geometry>
       </visual>
@@ -77,5 +77,5 @@
         <origin rpy="0 0 0" xyz="-0.061266 0.066842 0.004951"/>
         <geometry>
-          <mesh filename="package://gtu_polar_arm_description/meshes/gripper/finger_l.dae"/>
+          <mesh filename="package://polar_description/meshes/gripper/finger_l.dae"/>
         </geometry>
       </collision>
@@ -90,5 +90,5 @@
         <origin rpy="0 0 0" xyz="0.047804 0.066842 0.004951"/>
         <geometry>
-          <mesh filename="package://gtu_polar_arm_description/meshes/gripper/finger_r.dae"/>
+          <mesh filename="package://polar_description/meshes/gripper/finger_r.dae"/>
         </geometry>
       </visual>
@@ -96,5 +96,5 @@
         <origin rpy="0 0 0" xyz="0.047804 0.066842 0.004951"/>
         <geometry>
-          <mesh filename="package://gtu_polar_arm_description/meshes/gripper/finger_r.dae"/>
+          <mesh filename="package://polar_description/meshes/gripper/finger_r.dae"/>
         </geometry>
       </collision>

File: robots/polar.gazebo.xacro (robot description, xacro)
@@ -1,5 +1,5 @@
 <?xml version="1.0" encoding="utf-8"?>
 <robot xmlns:xacro="http://www.ros.org/wiki/xacro">
-    <xacro:macro name="gtu_polar_gazebo" params="robot_name">
+    <xacro:macro name="polar_gazebo" params="robot_name">
         <!-- Link0 -->
         <gazebo reference="${robot_name}_link0">

File: robots/polar.transmission.xacro (robot description, xacro)
@@ -1,5 +1,5 @@
 <?xml version="1.0" encoding="utf-8"?>
 <robot xmlns:xacro="http://www.ros.org/wiki/xacro">
-    <xacro:macro name="gtu_polar_transmission" params="robot_name">
+    <xacro:macro name="polar_transmission" params="robot_name">
         <!-- Load Gazebo lib and set the robot namespace -->
         <gazebo>

File: robots/polar_arm.xacro (robot description, xacro)
@@ -1,7 +1,7 @@
 <?xml version='1.0' encoding='utf-8'?>
-<robot xmlns:xacro="http://www.ros.org/wiki/xacro" name="gtu_polar">
+<robot xmlns:xacro="http://www.ros.org/wiki/xacro" name="polar">
   <!-- safety_distance: Minimum safety distance in [m] by which the collision volumes are expanded and which is enforced during robot motions -->
-  <!-- arm_id: Namespace of the gtu_polar arm. Serves to differentiate between arms in case of multiple instances. -->
-  <xacro:macro name="gtu_polar_arm" params="arm_id:='gtu_polar' description_pkg:='gtu_polar_arm_description' connected_to:='' xyz:='0 0 0' rpy:='0 0 0'">
+  <!-- arm_id: Namespace of the polar arm. Serves to differentiate between arms in case of multiple instances. -->
+  <xacro:macro name="polar_arm" params="arm_id:='polar' description_pkg:='polar_description' connected_to:='' xyz:='0 0 0' rpy:='0 0 0'">
     <xacro:unless value="${not connected_to}">
       <joint name="${arm_id}_joint_${connected_to}" type="fixed">
