Commit message: polar_description: - fix hand gazebo transmisson

File: robots/polar.transmission.xacro (robot description, xacro)
@@ -70,5 +70,5 @@
         </transmission>
         <!-- Hand -->
-        <transmission name="${robot_name}_hand_tran">
+        <transmission name="${robot_name}_hand_tran_1">
             <type>transmission_interface/SimpleTransmission</type>
             <joint name="${robot_name}_hand_joint1">
@@ -80,6 +80,36 @@
             </actuator>
         </transmission>
+        <transmission name="${robot_name}_hand_tran_2">
+            <type>transmission_interface/SimpleTransmission</type>
+            <joint name="${robot_name}_hand_joint2">
+                <hardwareInterface>hardware_interface/PositionJointInterface</hardwareInterface>
+            </joint>
+            <actuator name="${robot_name}_hand_motor_2">
+                <hardwareInterface>hardware_interface/PositionJointInterface</hardwareInterface>
+                <mechanicalReduction>1</mechanicalReduction>
+            </actuator>
+        </transmission>
+        <transmission name="${robot_name}_hand_tran_3">
+            <type>transmission_interface/SimpleTransmission</type>
+            <joint name="${robot_name}_finger_joint1">
+                <hardwareInterface>hardware_interface/PositionJointInterface</hardwareInterface>
+            </joint>
+            <actuator name="${robot_name}_hand_motor_3">
+                <hardwareInterface>hardware_interface/PositionJointInterface</hardwareInterface>
+                <mechanicalReduction>1</mechanicalReduction>
+            </actuator>
+        </transmission>
+        <transmission name="${robot_name}_hand_tran_4">
+            <type>transmission_interface/SimpleTransmission</type>
+            <joint name="${robot_name}_finger_joint2">
+                <hardwareInterface>hardware_interface/PositionJointInterface</hardwareInterface>
+            </joint>
+            <actuator name="${robot_name}_hand_motor_4">
+                <hardwareInterface>hardware_interface/PositionJointInterface</hardwareInterface>
+                <mechanicalReduction>1</mechanicalReduction>
+            </actuator>
+        </transmission>
         <!-- Mimic joints -->
-        <!-- <gazebo>
+        <gazebo>
             <plugin filename="libgazebo_mimic_joint_plugin.so" name="${robot_name}_hand_mimic_1">
                 <joint>${robot_name}_hand_joint2</joint>
@@ -100,5 +130,5 @@
                 <offset>0.0</offset>
             </plugin>
-        </gazebo> -->
+        </gazebo>
     </xacro:macro>
 </robot>

File: robots/polar_arm.xacro (robot description, xacro)
@@ -5,20 +5,14 @@
   <xacro:macro name="polar_arm" params="arm_id:='polar' description_pkg:='polar_description' connected_to:='' xyz:='0 0 0' rpy:='0 0 0'">
     <xacro:unless value="${not connected_to}">
-      <joint name="${arm_id}_joint_${connected_to}" type="fixed">
-        <parent link="${connected_to}"/>
-        <child link="${arm_id}_link0"/>
+      <joint name="virtual_joint" type="fixed">
+        <parent link="${connected_to}"/> <!-- world -->
+        <child link="${arm_id}_link0"/> <!-- base link -->
         <origin rpy="${rpy}" xyz="${xyz}"/>
       </joint>
     </xacro:unless>
-    <xacro:property name="joint_damping" value="0.0"/>
+    <xacro:property name="joint_damping" value="1.0"/>
     <xacro:property name="joint_friction" value="0.0"/>
     <xacro:property name="safety_k_position" value="100.0"/>
     <xacro:property name="safety_k_velocity" value="40.0"/>
-    <link name="world" />
-    <joint name="robot_to_world" type="fixed">
-      <parent link="world" />
-      <child link="${arm_id}_link0" />
-      <origin xyz="0.0 0.0 0.0" rpy="0.0 0.0 0.0" />
-    </joint>
     <link name="${arm_id}_link0">
       <visual>
@@ -65,5 +59,5 @@
       <child link="${arm_id}_link1"/>
       <axis xyz="-0.0048 0.0 1.0"/>
-      <limit effort="87" lower="${-1.2*pi}" upper="${1.2*pi}" velocity="2.1750"/>
+      <limit effort="200" lower="${-1.2*pi}" upper="${1.2*pi}" velocity="2.1750"/>
       <dynamics damping="${joint_damping}" friction="${joint_friction}"/>
     </joint>
@@ -93,5 +87,5 @@
       <child link="${arm_id}_link2"/>
       <axis xyz="-1.0 -0.0048 -0.0048"/>
-      <limit effort="87" lower="-0.96" upper="0.35" velocity="2.1750"/>
+      <limit effort="200" lower="-0.96" upper="0.35" velocity="2.1750"/>
       <dynamics damping="${joint_damping}" friction="${joint_friction}"/>
     </joint>
@@ -121,5 +115,5 @@
       <child link="${arm_id}_link3"/>
       <axis xyz="1.0 0.0048 0.0048"/>
-      <limit effort="87" lower="-0.26" upper="0.87" velocity="2.1750"/>
+      <limit effort="200" lower="-0.26" upper="0.87" velocity="2.1750"/>
       <dynamics damping="${joint_damping}" friction="${joint_friction}"/>
     </joint>
@@ -149,5 +143,5 @@
       <child link="${arm_id}_link4"/>
       <axis xyz="0.0048 -1.0 0.0"/>
-      <limit effort="87" lower="${-pi}" upper="${pi}" velocity="2.1750"/>
+      <limit effort="200" lower="${-pi}" upper="${pi}" velocity="2.1750"/>
       <dynamics damping="${joint_damping}" friction="${joint_friction}"/>
     </joint>
@@ -177,5 +171,5 @@
       <child link="${arm_id}_link5"/>
       <axis xyz="1.0 0.0048 0.0048"/>
-      <limit effort="12" lower="${-pi}" upper="0.96" velocity="2.6100"/>
+      <limit effort="100" lower="${-pi}" upper="0.96" velocity="2.6100"/>
       <dynamics damping="${joint_damping}" friction="${joint_friction}"/>
     </joint>
@@ -205,5 +199,5 @@
       <child link="${arm_id}_link6"/>
       <axis xyz="0.0048 -0.0 -1.0"/>
-      <limit effort="12" lower="${-pi}" upper="${pi}" velocity="2.6100"/>
+      <limit effort="100" lower="${-pi}" upper="${pi}" velocity="2.6100"/>
       <dynamics damping="${joint_damping}" friction="${joint_friction}"/>
     </joint>

File: robots/polar_arm_hand.urdf.xacro (robot description, xacro)
@@ -6,5 +6,6 @@
   <xacro:include filename="$(find polar_description)/robots/polar.gazebo.xacro"/>
   <xacro:include filename="$(find polar_description)/robots/polar.transmission.xacro"/>
-  <xacro:polar_arm/>
+  <link name="world" />
+  <xacro:polar_arm xyz="0 0 0" rpy="0 0 0" connected_to="world"/>
   <xacro:hand ns="polar" rpy="${pi/2} 0 0" xyz="-0.00675 -0.00964 -0.06152" connected_to="polar_link6"/>
   <xacro:polar_gazebo robot_name="$(arg robot_name)" />

Commit message: polar_description: - set safety limits - change gazebo control plugin

File: robots/polar.transmission.xacro (robot description, xacro)
@@ -2,9 +2,7 @@
 <robot xmlns:xacro="http://www.ros.org/wiki/xacro">
     <xacro:macro name="polar_transmission" params="robot_name">
-        <!-- Load Gazebo lib and set the robot namespace -->
+        <!-- (from ur_gazebo)  -->
         <gazebo>
-            <plugin name="gazebo_ros_control" filename="libgazebo_ros_control.so">
-                <robotNamespace>/${robot_name}</robotNamespace>
-            </plugin>
+            <plugin name="ros_control" filename="libgazebo_ros_control.so"></plugin>
         </gazebo>
         <!-- Polar arm -->

File: robots/polar_arm.xacro (robot description, xacro)
@@ -11,8 +11,9 @@
       </joint>
     </xacro:unless>
-    <xacro:property name="joint_damping" value="1.0"/>
+    <xacro:property name="joint_damping" value="0.0"/>
     <xacro:property name="joint_friction" value="0.0"/>
-    <xacro:property name="safety_k_position" value="100.0"/>
-    <xacro:property name="safety_k_velocity" value="40.0"/>
+    <xacro:property name="safety_k_position" value="20.0"/>
+    <xacro:property name="safety_k_velocity" value="0.0"/>
+    <xacro:property name="safety_pos_margin" value="0.15"/>
     <link name="${arm_id}_link0">
       <visual>
@@ -54,5 +55,5 @@
     </link>
     <joint name="${arm_id}_joint1" type="revolute">
-      <safety_controller k_position="${safety_k_position}" k_velocity="${safety_k_velocity}" soft_lower_limit="${-1.2*pi}" soft_upper_limit="${1.2*pi}"/>
+      <safety_controller k_position="${safety_k_position}" k_velocity="${safety_k_velocity}" soft_lower_limit="${-1.2*pi + safety_pos_margin}" soft_upper_limit="${1.2*pi - safety_pos_margin}"/>
       <origin rpy="0 0 0" xyz="-0.0005 0.0 0.095"/>
       <parent link="${arm_id}_link0"/>
@@ -82,5 +83,5 @@
     </link>
     <joint name="${arm_id}_joint2" type="revolute">
-      <safety_controller k_position="${safety_k_position}" k_velocity="${safety_k_velocity}" soft_lower_limit="-0.96" soft_upper_limit="0.35"/>
+      <safety_controller k_position="${safety_k_position}" k_velocity="${safety_k_velocity}" soft_lower_limit="${-0.96 + safety_pos_margin}" soft_upper_limit="${0.35 - safety_pos_margin}"/>
       <origin rpy="0 0 0" xyz="-0.0005 0.064 0.049"/>
       <parent link="${arm_id}_link1"/>
@@ -110,5 +111,5 @@
     </link>
     <joint name="${arm_id}_joint3" type="revolute">
-      <safety_controller k_position="${safety_k_position}" k_velocity="${safety_k_velocity}" soft_lower_limit="-0.26" soft_upper_limit="0.87"/>
+      <safety_controller k_position="${safety_k_position}" k_velocity="${safety_k_velocity}" soft_lower_limit="${-0.26 + safety_pos_margin}" soft_upper_limit="${0.87 - safety_pos_margin}"/>
       <origin rpy="0 0 0" xyz="-0.0014 -0.1437 0.4425"/>
       <parent link="${arm_id}_link2"/>
@@ -138,5 +139,5 @@
     </link>
     <joint name="${arm_id}_joint4" type="revolute">
-      <safety_controller k_position="${safety_k_position}" k_velocity="${safety_k_velocity}" soft_lower_limit="${-pi}" soft_upper_limit="${pi}"/>
+      <safety_controller k_position="${safety_k_position}" k_velocity="${safety_k_velocity}" soft_lower_limit="${-pi + safety_pos_margin}" soft_upper_limit="${pi - safety_pos_margin}"/>
       <origin rpy="0 0 0" xyz="0.0009 -0.1830 0.0"/>
       <parent link="${arm_id}_link3"/>
@@ -166,5 +167,5 @@
     </link>
     <joint name="${arm_id}_joint5" type="revolute">
-      <safety_controller k_position="${safety_k_position}" k_velocity="${safety_k_velocity}" soft_lower_limit="${-pi}" soft_upper_limit="0.96"/>
+      <safety_controller k_position="${safety_k_position}" k_velocity="${safety_k_velocity}" soft_lower_limit="${-pi + safety_pos_margin}" soft_upper_limit="${0.96 - safety_pos_margin}"/>
       <origin rpy="0 0 0" xyz="0.0007 -0.1515 0.0"/>
       <parent link="${arm_id}_link4"/>
@@ -194,5 +195,5 @@
     </link>
     <joint name="${arm_id}_joint6" type="revolute">
-      <safety_controller k_position="${safety_k_position}" k_velocity="${safety_k_velocity}" soft_lower_limit="${-pi}" soft_upper_limit="${pi}"/>
+      <safety_controller k_position="${safety_k_position}" k_velocity="${safety_k_velocity}" soft_lower_limit="${-pi + safety_pos_margin}" soft_upper_limit="${pi - safety_pos_margin}"/>
       <origin rpy="0 0 0" xyz="0.0008 -0.0 -0.1630"/>
       <parent link="${arm_id}_link5"/>
