Commit message: polar_description: round hand inertials

File: robots/hand.xacro (robot description, xacro)
@@ -23,4 +23,9 @@
         </geometry>
       </collision>
+      <inertial>
+        <origin rpy="0 0 0" xyz="0.006846 0.005366 -0.009625"/>
+        <mass value="1.2773"/>
+        <inertia ixx="0.0011" ixy="0.0" ixz="0.0" iyy="0.0006" iyz="0.0" izz="0.0015"/>
+      </inertial>
     </link>
     <link name="${ns}_outer_r">
@@ -37,4 +42,9 @@
         </geometry>
       </collision>
+      <inertial>
+        <origin rpy="0 0 0" xyz="-0.007134 -0.006305 -0.004655"/>
+        <mass value="0.0868"/>
+        <inertia ixx="0.0" ixy="0.0" ixz="0.0" iyy="0.0" iyz="-0.0" izz="0.0"/>
+      </inertial>
     </link>
     <link name="${ns}_outer_l">
@@ -51,4 +61,9 @@
         </geometry>
       </collision>
+      <inertial>
+        <origin rpy="0 0 0" xyz="0.006975 -0.006230 -0.004655"/>
+        <mass value="0.0877"/>
+        <inertia ixx="0.0" ixy="0.0" ixz="-0.0" iyy="0.0" iyz="0.0" izz="0.0"/>
+      </inertial>
     </link>
     <link name="${ns}_finger_l">
@@ -65,4 +80,9 @@
         </geometry>
       </collision>
+      <inertial>
+        <origin rpy="0 0 0" xyz="0.006607 -0.028924 -0.004655"/>
+        <mass value="0.7779"/>
+        <inertia ixx="0.0009" ixy="0.0" ixz="-0.0" iyy="0.0003" iyz="0.0" izz="0.0009"/>
+      </inertial>
     </link>
     <link name="${ns}_finger_r">
@@ -79,4 +99,9 @@
         </geometry>
       </collision>
+      <inertial>
+        <origin rpy="0 0 0" xyz="-0.006607 -0.028924 -0.004655"/>
+        <mass value="0.7779"/>
+        <inertia ixx="0.0009" ixy="0.0" ixz="0.0" iyy="0.0003" iyz="0.0" izz="0.0009"/>
+      </inertial>
     </link>
     <joint name="${ns}_hand_joint2" type="continuous">

Commit message: polar_description: - convert hand mimic joints to revolute - add hand mimics transmission as template - generate gazebo urdf

File: robots/hand.xacro (robot description, xacro)
@@ -105,5 +105,5 @@
       </inertial>
     </link>
-    <joint name="${ns}_hand_joint2" type="continuous">
+    <joint name="${ns}_hand_joint2" type="revolute">
       <origin rpy="0 0 0" xyz="-0.011889 -0.027594 -0.004951"/>
       <parent link="${ns}_hand"/>
@@ -111,4 +111,5 @@
       <axis xyz="0.0 -0.0 -1.0"/>
       <mimic joint="${ns}_hand_joint1" multiplier="-1.0"/>
+      <limit effort="100" lower="-0.74002" upper="0.827286" velocity="100"/>
     </joint>
     <joint name="${ns}_hand_joint1" type="revolute">
@@ -119,12 +120,13 @@
       <limit effort="100" lower="-0.827286" upper="0.74002" velocity="100"/>
     </joint>
-    <joint name="${ns}_finger_joint1" type="continuous">
+    <joint name="${ns}_finger_joint1" type="revolute">
       <origin rpy="0 0 0" xyz="0.035915 -0.039248 0.0"/>
       <parent link="${ns}_outer_l"/>
       <child link="${ns}_finger_l"/>
       <axis xyz="-0.0 -0.0 -1.0"/>
-      <mimic joint="${ns}_finger_joint2"/>
+      <mimic joint="${ns}_hand_joint1" multiplier="-1.0"/>
+      <limit effort="100" lower="-0.74002" upper="0.827286" velocity="100"/>
     </joint>
-    <joint name="${ns}_finger_joint2" type="continuous">
+    <joint name="${ns}_finger_joint2" type="revolute">
       <origin rpy="0 0 0" xyz="-0.035915 -0.039248 0.0"/>
       <parent link="${ns}_outer_r"/>
@@ -132,4 +134,5 @@
       <axis xyz="0.0 0.0 1.0"/>
       <mimic joint="${ns}_hand_joint1" multiplier="-1.0"/>
+      <limit effort="100" lower="-0.74002" upper="0.827286" velocity="100"/>
     </joint>
   </xacro:macro>

File: robots/polar.transmission.xacro (robot description, xacro)
@@ -8,11 +8,12 @@
             </plugin>
         </gazebo>
+        <!-- Polar arm -->
         <transmission name="${robot_name}_tran_1">
             <type>transmission_interface/SimpleTransmission</type>
             <joint name="${robot_name}_joint1">
-                <hardwareInterface>hardware_interface/EffortJointInterface</hardwareInterface> <!-- Effort type is for gazebo -->
+                <hardwareInterface>hardware_interface/PositionJointInterface</hardwareInterface>
             </joint>
             <actuator name="${robot_name}_motor_1">
-                <hardwareInterface>hardware_interface/EffortJointInterface</hardwareInterface>
+                <hardwareInterface>hardware_interface/PositionJointInterface</hardwareInterface>
                 <mechanicalReduction>1</mechanicalReduction>
             </actuator>
@@ -21,8 +22,8 @@
             <type>transmission_interface/SimpleTransmission</type>
             <joint name="${robot_name}_joint2">
-                <hardwareInterface>hardware_interface/EffortJointInterface</hardwareInterface>
+                <hardwareInterface>hardware_interface/PositionJointInterface</hardwareInterface>
             </joint>
             <actuator name="${robot_name}_motor_2">
-                <hardwareInterface>hardware_interface/EffortJointInterface</hardwareInterface>
+                <hardwareInterface>hardware_interface/PositionJointInterface</hardwareInterface>
                 <mechanicalReduction>1</mechanicalReduction>
             </actuator>
@@ -31,8 +32,8 @@
             <type>transmission_interface/SimpleTransmission</type>
             <joint name="${robot_name}_joint3">
-                <hardwareInterface>hardware_interface/EffortJointInterface</hardwareInterface>
+                <hardwareInterface>hardware_interface/PositionJointInterface</hardwareInterface>
             </joint>
             <actuator name="${robot_name}_motor_3">
-                <hardwareInterface>hardware_interface/EffortJointInterface</hardwareInterface>
+                <hardwareInterface>hardware_interface/PositionJointInterface</hardwareInterface>
                 <mechanicalReduction>1</mechanicalReduction>
             </actuator>
@@ -41,8 +42,8 @@
             <type>transmission_interface/SimpleTransmission</type>
             <joint name="${robot_name}_joint4">
-                <hardwareInterface>hardware_interface/EffortJointInterface</hardwareInterface>
+                <hardwareInterface>hardware_interface/PositionJointInterface</hardwareInterface>
             </joint>
             <actuator name="${robot_name}_motor_4">
-                <hardwareInterface>hardware_interface/EffortJointInterface</hardwareInterface>
+                <hardwareInterface>hardware_interface/PositionJointInterface</hardwareInterface>
                 <mechanicalReduction>1</mechanicalReduction>
             </actuator>
@@ -51,8 +52,8 @@
             <type>transmission_interface/SimpleTransmission</type>
             <joint name="${robot_name}_joint5">
-                <hardwareInterface>hardware_interface/EffortJointInterface</hardwareInterface>
+                <hardwareInterface>hardware_interface/PositionJointInterface</hardwareInterface>
             </joint>
             <actuator name="${robot_name}_motor_5">
-                <hardwareInterface>hardware_interface/EffortJointInterface</hardwareInterface>
+                <hardwareInterface>hardware_interface/PositionJointInterface</hardwareInterface>
                 <mechanicalReduction>1</mechanicalReduction>
             </actuator>
@@ -61,21 +62,43 @@
             <type>transmission_interface/SimpleTransmission</type>
             <joint name="${robot_name}_joint6">
-                <hardwareInterface>hardware_interface/EffortJointInterface</hardwareInterface>
+                <hardwareInterface>hardware_interface/PositionJointInterface</hardwareInterface>
             </joint>
             <actuator name="${robot_name}_motor_6">
-                <hardwareInterface>hardware_interface/EffortJointInterface</hardwareInterface>
+                <hardwareInterface>hardware_interface/PositionJointInterface</hardwareInterface>
                 <mechanicalReduction>1</mechanicalReduction>
             </actuator>
         </transmission>
+        <!-- Hand -->
         <transmission name="${robot_name}_hand_tran">
             <type>transmission_interface/SimpleTransmission</type>
             <joint name="${robot_name}_hand_joint1">
-                <hardwareInterface>hardware_interface/EffortJointInterface</hardwareInterface>
+                <hardwareInterface>hardware_interface/PositionJointInterface</hardwareInterface>
             </joint>
-            <actuator name="${robot_name}_hand_motor">
-                <hardwareInterface>hardware_interface/EffortJointInterface</hardwareInterface>
+            <actuator name="${robot_name}_hand_motor_1">
+                <hardwareInterface>hardware_interface/PositionJointInterface</hardwareInterface>
                 <mechanicalReduction>1</mechanicalReduction>
             </actuator>
         </transmission>
+        <!-- Mimic joints -->
+        <!-- <gazebo>
+            <plugin filename="libgazebo_mimic_joint_plugin.so" name="${robot_name}_hand_mimic_1">
+                <joint>${robot_name}_hand_joint2</joint>
+                <mimicJoint>${robot_name}_hand_joint1</mimicJoint>
+                <multiplier>-1.0</multiplier>
+                <offset>0.0</offset>
+            </plugin>
+            <plugin filename="libgazebo_mimic_joint_plugin.so" name="${robot_name}_hand_mimic_2">
+                <joint>${robot_name}_finger_joint1</joint>
+                <mimicJoint>${robot_name}_hand_joint1</mimicJoint>
+                <multiplier>-1.0</multiplier>
+                <offset>0.0</offset>
+            </plugin>
+            <plugin filename="libgazebo_mimic_joint_plugin.so" name="${robot_name}_hand_mimic_3">
+                <joint>${robot_name}_finger_joint2</joint>
+                <mimicJoint>${robot_name}_hand_joint1</mimicJoint>
+                <multiplier>-1.0</multiplier>
+                <offset>0.0</offset>
+            </plugin>
+        </gazebo> -->
     </xacro:macro>
 </robot>

Commit message: polar_description: - real joint limits - new home position - add rover to link0

File: robots/hand.xacro (robot description, xacro)
@@ -111,5 +111,5 @@
       <axis xyz="0.0 -0.0 -1.0"/>
       <mimic joint="${ns}_hand_joint1" multiplier="-1.0"/>
-      <limit effort="100" lower="-0.74002" upper="0.827286" velocity="100"/>
+      <limit effort="100" lower="-0.74002" upper="0.827286" velocity="6.5449"/>
     </joint>
     <joint name="${ns}_hand_joint1" type="revolute">
@@ -118,5 +118,5 @@
       <child link="${ns}_outer_l"/>
       <axis xyz="0.0 -0.0 -1.0"/>
-      <limit effort="100" lower="-0.827286" upper="0.74002" velocity="100"/>
+      <limit effort="100" lower="-0.827286" upper="0.74002" velocity="6.5449"/>
     </joint>
     <joint name="${ns}_finger_joint1" type="revolute">
@@ -126,5 +126,5 @@
       <axis xyz="-0.0 -0.0 -1.0"/>
       <mimic joint="${ns}_hand_joint1" multiplier="-1.0"/>
-      <limit effort="100" lower="-0.74002" upper="0.827286" velocity="100"/>
+      <limit effort="100" lower="-0.74002" upper="0.827286" velocity="6.5449"/>
     </joint>
     <joint name="${ns}_finger_joint2" type="revolute">
@@ -134,5 +134,5 @@
       <axis xyz="0.0 0.0 1.0"/>
       <mimic joint="${ns}_hand_joint1" multiplier="-1.0"/>
-      <limit effort="100" lower="-0.74002" upper="0.827286" velocity="100"/>
+      <limit effort="100" lower="-0.74002" upper="0.827286" velocity="6.5449"/>
     </joint>
   </xacro:macro>

File: robots/polar_arm.xacro (robot description, xacro)
@@ -15,5 +15,5 @@
     <xacro:property name="safety_k_position" value="20.0"/>
     <xacro:property name="safety_k_velocity" value="0.0"/>
-    <xacro:property name="safety_pos_margin" value="0.15"/>
+    <xacro:property name="safety_pos_margin" value="0.0"/>
     <link name="${arm_id}_link0">
       <visual>
@@ -60,5 +60,5 @@
       <child link="${arm_id}_link1"/>
       <axis xyz="-0.0048 0.0 1.0"/>
-      <limit effort="200" lower="${-1.2*pi}" upper="${1.2*pi}" velocity="2.1750"/>
+      <limit effort="100" lower="${-1.2*pi}" upper="${1.2*pi}" velocity="0.1286"/>
       <dynamics damping="${joint_damping}" friction="${joint_friction}"/>
     </joint>
@@ -83,10 +83,10 @@
     </link>
     <joint name="${arm_id}_joint2" type="revolute">
-      <safety_controller k_position="${safety_k_position}" k_velocity="${safety_k_velocity}" soft_lower_limit="${-0.96 + safety_pos_margin}" soft_upper_limit="${0.35 - safety_pos_margin}"/>
-      <origin rpy="0 0 0" xyz="-0.0005 0.064 0.049"/>
+      <safety_controller k_position="${safety_k_position}" k_velocity="${safety_k_velocity}" soft_lower_limit="${-1.2968 + safety_pos_margin}" soft_upper_limit="${0 - safety_pos_margin}"/>
+      <origin rpy="-0.3813 0 0" xyz="-0.0005 0.064 0.049"/>
       <parent link="${arm_id}_link1"/>
       <child link="${arm_id}_link2"/>
       <axis xyz="-1.0 -0.0048 -0.0048"/>
-      <limit effort="200" lower="-0.96" upper="0.35" velocity="2.1750"/>
+      <limit effort="100" lower="-1.2968" upper="0" velocity="0.1071"/>
       <dynamics damping="${joint_damping}" friction="${joint_friction}"/>
     </joint>
@@ -111,10 +111,10 @@
     </link>
     <joint name="${arm_id}_joint3" type="revolute">
-      <safety_controller k_position="${safety_k_position}" k_velocity="${safety_k_velocity}" soft_lower_limit="${-0.26 + safety_pos_margin}" soft_upper_limit="${0.87 - safety_pos_margin}"/>
-      <origin rpy="0 0 0" xyz="-0.0014 -0.1437 0.4425"/>
+      <safety_controller k_position="${safety_k_position}" k_velocity="${safety_k_velocity}" soft_lower_limit="${0 + safety_pos_margin}" soft_upper_limit="${1.1537 - safety_pos_margin}"/>
+      <origin rpy="-0.3951 0 0" xyz="-0.0014 -0.1437 0.4425"/>
       <parent link="${arm_id}_link2"/>
       <child link="${arm_id}_link3"/>
       <axis xyz="1.0 0.0048 0.0048"/>
-      <limit effort="200" lower="-0.26" upper="0.87" velocity="2.1750"/>
+      <limit effort="100" lower="0" upper="1.1537" velocity="0.0637"/>
       <dynamics damping="${joint_damping}" friction="${joint_friction}"/>
     </joint>
@@ -144,5 +144,5 @@
       <child link="${arm_id}_link4"/>
       <axis xyz="0.0048 -1.0 0.0"/>
-      <limit effort="200" lower="${-pi}" upper="${pi}" velocity="2.1750"/>
+      <limit effort="100" lower="${-pi}" upper="${pi}" velocity="0.8722"/>
       <dynamics damping="${joint_damping}" friction="${joint_friction}"/>
     </joint>
@@ -167,10 +167,10 @@
     </link>
     <joint name="${arm_id}_joint5" type="revolute">
-      <safety_controller k_position="${safety_k_position}" k_velocity="${safety_k_velocity}" soft_lower_limit="${-pi + safety_pos_margin}" soft_upper_limit="${0.96 - safety_pos_margin}"/>
-      <origin rpy="0 0 0" xyz="0.0007 -0.1515 0.0"/>
+      <safety_controller k_position="${safety_k_position}" k_velocity="${safety_k_velocity}" soft_lower_limit="${-3.6530 + safety_pos_margin}" soft_upper_limit="${0 - safety_pos_margin}"/>
+      <origin rpy="0.3333 0 0" xyz="0.0007 -0.1515 0.0"/>
       <parent link="${arm_id}_link4"/>
       <child link="${arm_id}_link5"/>
       <axis xyz="1.0 0.0048 0.0048"/>
-      <limit effort="100" lower="${-pi}" upper="0.96" velocity="2.6100"/>
+      <limit effort="100" lower="-3.6530" upper="0" velocity="0.1626"/>
       <dynamics damping="${joint_damping}" friction="${joint_friction}"/>
     </joint>
@@ -200,5 +200,5 @@
       <child link="${arm_id}_link6"/>
       <axis xyz="0.0048 -0.0 -1.0"/>
-      <limit effort="100" lower="${-pi}" upper="${pi}" velocity="2.6100"/>
+      <limit effort="100" lower="${-pi}" upper="${pi}" velocity="0.8845"/>
       <dynamics damping="${joint_damping}" friction="${joint_friction}"/>
     </joint>
