Commit message: polar_description: - new gripper

File: robots/hand.xacro (robot description, xacro)
@@ -10,4 +10,5 @@
       </joint>
     </xacro:unless>
+    <xacro:property name="limit" value="${60 * pi / 180}"/>
     <link name="${ns}_hand">
       <visual>
@@ -24,12 +25,12 @@
       </collision>
       <inertial>
-        <origin rpy="0 0 0" xyz="0.006846 0.005366 -0.009625"/>
-        <mass value="1.2773"/>
-        <inertia ixx="0.0011" ixy="0.0" ixz="0.0" iyy="0.0006" iyz="0.0" izz="0.0015"/>
+        <origin rpy="0 0 0" xyz="0.006733 -0.006163 -0.009538"/>
+        <mass value="2.3427"/>
+        <inertia ixx="0.0028" ixy="0" ixz="-0.0004" iyy="0.0023" iyz="0" izz="0.0035"/>
       </inertial>
     </link>
     <link name="${ns}_outer_l">
       <visual>
-        <origin rpy="0 0 0" xyz="-0.025351 0.027594 0.004951"/>
+        <origin rpy="0 0 0" xyz="-0.040231 0.024653 0.007426"/>
         <geometry>
           <mesh filename="package://polar_description/meshes/gripper/outer_l.dae"/>
@@ -37,5 +38,5 @@
       </visual>
       <collision>
-        <origin rpy="0 0 0" xyz="-0.025351 0.027594 0.004951"/>
+        <origin rpy="0 0 0" xyz="-0.040231 0.024653 0.007426"/>
         <geometry>
           <mesh filename="package://polar_description/meshes/gripper/outer_l.dae"/>
@@ -43,12 +44,12 @@
       </collision>
       <inertial>
-        <origin rpy="0 0 0" xyz="0.006975 -0.006230 -0.004655"/>
-        <mass value="0.0877"/>
-        <inertia ixx="0.0" ixy="0.0" ixz="-0.0" iyy="0.0" iyz="0.0" izz="0.0"/>
+        <origin rpy="0 0 0" xyz="0 -0.013601 -0.0020100"/>
+        <mass value="0.0589"/>
+        <inertia ixx="0" ixy="-0.0" ixz="0.0" iyy="0" iyz="0.0" izz="0"/>
       </inertial>
     </link>
     <link name="${ns}_outer_r">
       <visual>
-        <origin rpy="0 0 0" xyz="0.011889 0.027594 0.004951"/>
+        <origin rpy="0 0 0" xyz="0.026768 0.024652 0.011626"/>
         <geometry>
           <mesh filename="package://polar_description/meshes/gripper/outer_r.dae"/>
@@ -56,5 +57,5 @@
       </visual>
       <collision>
-        <origin rpy="0 0 0" xyz="0.011889 0.027594 0.004951"/>
+        <origin rpy="0 0 0" xyz="0.026768 0.024652 0.011626"/>
         <geometry>
           <mesh filename="package://polar_description/meshes/gripper/outer_r.dae"/>
@@ -62,12 +63,12 @@
       </collision>
       <inertial>
-        <origin rpy="0 0 0" xyz="-0.007134 -0.006305 -0.004655"/>
-        <mass value="0.0868"/>
-        <inertia ixx="0.0" ixy="0.0" ixz="0.0" iyy="0.0" iyz="-0.0" izz="0.0"/>
+        <origin rpy="0 0 0" xyz="0 -0.013627 0.002093"/>
+        <mass value="0.058776"/>
+        <inertia ixx="0" ixy="-0.0" ixz="-0.0" iyy="0" iyz="0.0" izz="0"/>
       </inertial>
     </link>
     <link name="${ns}_finger_l">
       <visual>
-        <origin rpy="0 0 0" xyz="-0.061266 0.066842 0.004951"/>
+        <origin rpy="0 0 0" xyz="-0.040231 0.069653 0.013526"/>
         <geometry>
           <mesh filename="package://polar_description/meshes/gripper/finger_l.dae"/>
@@ -75,5 +76,5 @@
       </visual>
       <collision>
-        <origin rpy="0 0 0" xyz="-0.061266 0.066842 0.004951"/>
+        <origin rpy="0 0 0" xyz="-0.040231 0.069653 0.013526"/>
         <geometry>
           <mesh filename="package://polar_description/meshes/gripper/finger_l.dae"/>
@@ -81,12 +82,12 @@
       </collision>
       <inertial>
-        <origin rpy="0 0 0" xyz="0.006607 -0.028924 -0.004655"/>
-        <mass value="0.7779"/>
-        <inertia ixx="0.0009" ixy="0.0" ixz="-0.0" iyy="0.0003" iyz="0.0" izz="0.0009"/>
+        <origin rpy="0 0 0" xyz="-0.010571 -0.034963 0.004031"/>
+        <mass value="0.5436"/>
+        <inertia ixx="0.0004" ixy="0" ixz="-0.0" iyy="0.0001" iyz="0" izz="0.0004"/>
       </inertial>
     </link>
     <link name="${ns}_finger_r">
       <visual>
-        <origin rpy="0 0 0" xyz="0.047804 0.066842 0.004951"/>
+        <origin rpy="0 0 0" xyz="0.026768 0.069652 0.013526"/>
         <geometry>
           <mesh filename="package://polar_description/meshes/gripper/finger_r.dae"/>
@@ -94,5 +95,5 @@
       </visual>
       <collision>
-        <origin rpy="0 0 0" xyz="0.047804 0.066842 0.004951"/>
+        <origin rpy="0 0 0" xyz="0.026768 0.069652 0.013526"/>
         <geometry>
           <mesh filename="package://polar_description/meshes/gripper/finger_r.dae"/>
@@ -100,39 +101,39 @@
       </collision>
       <inertial>
-        <origin rpy="0 0 0" xyz="-0.006607 -0.028924 -0.004655"/>
-        <mass value="0.7779"/>
-        <inertia ixx="0.0009" ixy="0.0" ixz="0.0" iyy="0.0003" iyz="0.0" izz="0.0009"/>
+        <origin rpy="0 0 0" xyz="0.010571 -0.034962 0.003969"/>
+        <mass value="0.5436"/>
+        <inertia ixx="0.0004" ixy="0" ixz="-0.0" iyy="0.0001" iyz="0" izz="0.0004"/>
       </inertial>
     </link>
     <joint name="${ns}_hand_joint2" type="revolute">
-      <origin rpy="0 0 0" xyz="-0.011889 -0.027594 -0.004951"/>
+      <origin rpy="0 0 0" xyz="-0.026768 -0.024652 -0.011626"/>
       <parent link="${ns}_hand"/>
       <child link="${ns}_outer_r"/>
-      <axis xyz="0.0 -0.0 -1.0"/>
-      <mimic joint="${ns}_hand_joint1" multiplier="-1.0"/>
-      <limit effort="100" lower="-0.74002" upper="0.827286" velocity="6.5449"/>
+      <axis xyz="-0.0 0.0 1.0"/>
+      <mimic joint="${ns}_hand_joint1" multiplier="1.0"/>
+      <limit effort="100" lower="${-limit}" upper="0" velocity="6.5449"/>
     </joint>
     <joint name="${ns}_hand_joint1" type="revolute">
-      <origin rpy="0 0 0" xyz="0.025351 -0.027594 -0.004951"/>
+      <origin rpy="0 0 0" xyz="0.040231 -0.024653 -0.007426"/>
       <parent link="${ns}_hand"/>
       <child link="${ns}_outer_l"/>
       <axis xyz="0.0 -0.0 -1.0"/>
-      <limit effort="100" lower="-0.827286" upper="0.74002" velocity="6.5449"/>
+      <limit effort="100" lower="${-limit}" upper="0" velocity="6.5449"/>
     </joint>
     <joint name="${ns}_finger_joint1" type="revolute">
-      <origin rpy="0 0 0" xyz="0.035915 -0.039248 0.0"/>
+      <origin rpy="0 0 0" xyz="0.0 -0.045 -0.0061"/>
       <parent link="${ns}_outer_l"/>
       <child link="${ns}_finger_l"/>
-      <axis xyz="-0.0 -0.0 -1.0"/>
+      <axis xyz="0.0 -0.0 -1.0"/>
       <mimic joint="${ns}_hand_joint1" multiplier="-1.0"/>
-      <limit effort="100" lower="-0.74002" upper="0.827286" velocity="6.5449"/>
+      <limit effort="100" lower="0" upper="${limit}" velocity="6.5449"/>
     </joint>
     <joint name="${ns}_finger_joint2" type="revolute">
-      <origin rpy="0 0 0" xyz="-0.035915 -0.039248 0.0"/>
+      <origin rpy="0 0 0" xyz="0.0 -0.045 -0.0019"/>
       <parent link="${ns}_outer_r"/>
       <child link="${ns}_finger_r"/>
-      <axis xyz="0.0 0.0 1.0"/>
-      <mimic joint="${ns}_hand_joint1" multiplier="-1.0"/>
-      <limit effort="100" lower="-0.74002" upper="0.827286" velocity="6.5449"/>
+      <axis xyz="0.0 -0.0 -1.0"/>
+      <mimic joint="${ns}_hand_joint1" multiplier="1.0"/>
+      <limit effort="100" lower="${-limit}" upper="0" velocity="6.5449"/>
     </joint>
   </xacro:macro>

File: robots/polar_arm.xacro (robot description, xacro)
@@ -168,9 +168,9 @@
     <joint name="${arm_id}_joint5" type="revolute">
       <safety_controller k_position="${safety_k_position}" k_velocity="${safety_k_velocity}" soft_lower_limit="${-3.6530 + safety_pos_margin}" soft_upper_limit="${0 - safety_pos_margin}"/>
-      <origin rpy="0.3333 0 0" xyz="0.0007 -0.1515 0.0"/>
+      <origin rpy="0.3333 0 0" xyz="0.0007 -0.1515 0.0"/> <!-- -1 derece -->
       <parent link="${arm_id}_link4"/>
       <child link="${arm_id}_link5"/>
       <axis xyz="1.0 0.0048 0.0048"/>
-      <limit effort="100" lower="-3.6530" upper="0" velocity="0.1626"/>
+      <limit effort="100" lower="-3.6530" upper="0" velocity="0.1626"/> <!-- lower +1 derece -->
       <dynamics damping="${joint_damping}" friction="${joint_friction}"/>
     </joint>
